File: FabOS_MB/ethernet.kicad_sch (KiCad schematic)
At the start: 4 parts, among them J3 RJ45, U7 CND-tek B1601S, U8 LAN8742A, U9 USBLC6-4SC6

Commit message: push
Other:
- moved on the sheet: J3, U7
Changed lines of the file:
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@@
 	(symbol
 		(lib_id "Librairie_MB:CND-tek_B1601S")
-		(at 187.325 63.5 0)
+		(at 190.5 63.5 0)
 		(unit 1)
 		(exclude_from_sim no)
@@
 		(dnp no)
 		(property "Reference" "U7"
-			(at 187.6425 40.64 0)
+			(at 190.8175 40.64 0)
 			(effects
 				(font
@@
 		)
 		(property "Value" "CND-tek B1601S"
-			(at 187.6425 43.18 0)
+			(at 190.8175 43.18 0)
 			(effects
 				(font
@@
 		)
 		(property "Footprint" "Librairie_MB:CND-Tek B1601S"
-			(at 187.325 63.5 0)
+			(at 190.5 63.5 0)
 			(effects
 				(font
@@
 		)
 		(property "Datasheet" "https://www.lcsc.com/datasheet/lcsc_datasheet_2405301629_CND-tek-B1601S_C510548.pdf"
-			(at 187.96 85.725 0)
+			(at 191.135 85.725 0)
 			(effects
 				(font
@@
 		)
 		(property "Description" "Transformateur Ethernet"
-			(at 188.595 61.595 0)
+			(at 191.77 61.595 0)
 			(effects
 				(font
@@
 		)
 		(property "MPN" "B1601S"
-			(at 187.325 63.5 0)
+			(at 190.5 63.5 0)
 			(effects
 				(font
@@
 		)
 		(property "LCSC" "C510548"
-			(at 187.071 84.328 0)
+			(at 190.246 84.328 0)
 			(effects
 				(font
@@
 	(symbol
 		(lib_id "Connector:RJ45")
-		(at 264.16 62.23 180)
+		(at 261.62 52.07 180)
 		(unit 1)
 		(exclude_from_sim no)
@@
 		(fields_autoplaced yes)
 		(property "Reference" "J3"
-			(at 261.9375 46.99 0)
+			(at 259.3975 36.83 0)
 			(effects
 				(font
@@
 		)
 		(property "Value" "RJ45"
-			(at 261.9375 49.53 0)
+			(at 259.3975 39.37 0)
 			(effects
 				(font
@@
 		)
 		(property "Footprint" "Librairie_MB:HC-RJ45-5JAS-1-5-01"
-			(at 263.525 79.375 0)
+			(at 260.985 69.215 0)
 			(effects
 				(font
@@
 		)
 		(property "Datasheet" "https://www.lcsc.com/datasheet/lcsc_datasheet_2401121837_HCTL-HC-RJ45-5JAS-1-5-01_C20417896.pdf"
-			(at 262.255 76.835 0)
+			(at 259.715 66.675 0)
 			(effects
 				(font
@@
 		)
 		(property "Description" "RJ connector, 8P8C (8 positions 8 connected)"
-			(at 264.16 46.99 0)
-			(effects
-				(font
+			(at 261.62 36.83 0)
+			(effects
+				(font
