File: FabOS_MB/ethernet.kicad_sch (KiCad schematic)
At the start: 43 parts, among them J1 RJ45, U3 LAN8742A, U4 USBLC6-4SC6, U5 CND-tek B1601S, Y1 Crystal_GND24

Commit message: update pcb
Connections:
- net RXCT: now reaches R19.1, U5.10 (RXCT)
- net RX+: now reaches J1.3 (RX+), U5.11 (RX+)
- net TX-: now reaches J1.2 (TX-), U5.14 (TX-)
- net TXCT: now reaches R20.1, U5.15 (TXCT)
- net TX+: now reaches J1.1 (TX+), U5.16 (TX+)
- net RX-: now reaches J1.6 (RX-), U5.9 (RX-)
- net Led 2 renamed LED2+
- net Led1 renamed LED1+
Other:
- note added: "2 Label pour le meme net, il faut faire un choix"
- note added: "C'est un quartz ou un oscillateur ?"
- note added: "ERREUR ?"
- note added: "Le NRST ne doit pas être le même que celui du processeur, renommer le NRST du PHY en NRST_LAN8742A et le relier à un GPIO du stm32"
- moved on the sheet: C10, C11, C12, C16, C17, JP1, R11, R12, R13, R18, R4, R5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
