File: FabOS_MB/_autosave-FabOS_MB.kicad_sch (KiCad schematic)
At the start: 2 parts, among them U1 STM32F407VETx

Commit message: Maj 5V
Connections:
- net USART3_RX: no longer names the net of U1.56 (PD9)
- net USART3_TX: no longer names the net of U1.47 (PB10)
Other:
- note removed: "Je suis incapable de savoir si le branchement de l'USB est cohérent"
Changed lines of the file:
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@@
-	(wire
-		(pts
-			(xy 76.2 100.33) (xy 72.39 100.33)
-		)
-		(stroke
-			(width 0)
-			(type default)
-		)
-	)
 	(wire
 		(pts
@@
 		)
 	)
-	(text "Je suis incapable de savoir si le branchement de l'USB est cohérent\n"
-		(exclude_from_sim no)
-		(at 147.574 122.936 0)
-		(effects
-			(font
-				(size 1.27 1.27)
-			)
-		)
-	)
 	(text "Comment gérer le boot ?\nUSART ou OTG_deviceonly ?\n"
 		(exclude_from_sim no)
@@
 		)
 	)
-	(label "USART3_TX"
-		(at 76.2 100.33 0)
-		(fields_autoplaced yes)
-		(effects
-			(font
-				(size 1.27 1.27)
-			)
-			(justify left bottom)
-		)
-	)
 	(label "USART1_RX"
 		(at 275.59 62.23 0)
@@
 		)
 	)
+	(label "USB_OTG_DM"
+		(at 166.37 111.76 0)
+		(fields_autoplaced yes)
+		(effects
+			(font
+				(size 1.27 1.27)
+			)
+			(justify left bottom)
+		)
+	)
 	(label "ETH_MDC"
 		(at 76.2 120.65 0)
@@
 		)
 	)
-	(label "USART3_RX"
-		(at 26.67 120.65 180)
-		(fields_autoplaced yes)
-		(effects
-			(font
-				(size 1.27 1.27)
-			)
-			(justify right bottom)
-		)
-	)
 	(label "NRST"
 		(at 26.67 31.75 180)
@@
 		)
 	)
-	(label "USART3_RX"
-		(at 166.37 105.41 0)
-		(fields_autoplaced yes)
-		(effects
-			(font
-				(size 1.27 1.27)
-			)
-			(justify left bottom)
-		)
-	)
-	(label "USART3_TX"
-		(at 166.37 111.76 0)
-		(fields_autoplaced yes)
-		(effects
-			(font
-				(size 1.27 1.27)
-			)
-			(justify left bottom)
-		)
-	)
 	(label "ETH_TXD0"
 		(at 113.03 69.85 180)
@@
 	(label "ETH_TXD1"
 		(at 76.2 107.95 0)
+		(fields_autoplaced yes)
+		(effects
+			(font
+				(size 1.27 1.27)
+			)
+			(justify left bottom)
+		)
+	)
+	(label "USB_OTG_FS_DP"
+		(at 166.37 105.41 0)
 		(fields_autoplaced yes)
 		(effects
@@
 			)
 		)
-		(property "Value" "+3.3V"
+		(property "Value" "+5V"
 			(at 123.19 109.2199 90)
 			(effects
