File: FabOS_MB/switch.kicad_sch (KiCad schematic)
At the start: 2 parts, among them Q1 NMOS, U5 HF3F-L 12-1ZL1T

Commit message: jsp ce que je fais
mais j'espère que ça fonctionne
Parts:
- added Q2, Q3, Q4: NMOS, symbol Simulation_SPICE:NMOS
- added R24, R25, R26, R27: 22, Resistor_SMD:R_0402_1005Metric, symbol Device:R_Small
Connections:
- net at Q1.1 (D): now also U5.1 (set_+), Q4.1 (D)
- net at Q1.2 (G): now also R24.1
- net GND: now reaches Q1.3 (S)
- net GND: now also Q2.3 (S)
- net at U5.2 (reset_+): now also Q2.1 (D), Q3.1 (D)
- net 230 V entrée: now reaches U5.L (Vin)
- net 230 V sortie: now reaches U5.L1 (Vout1)
- net Earth: now reaches U5.L2 (Vout2)
- new net: Q2.2 (G), R27.2
- new net: Q3.2 (G), R26.1
- new net: Q4.2 (G), R25.2
- new net 12V: Q3.3 (S), Q4.3 (S)
- new net reset: R25.1, R27.1
- new net set: R24.2, R26.2
Other:
- moved on the sheet: Q1

Commit message: verif
Other:
- note added: "chgmt composants en 5,5 V et rajout pont H pour entree"
- note added: "je sais pas si ça marche c'est la merde"
Changed lines of the file:
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@@
 	)
 	(junction
-		(at 140.97 86.36)
+		(at 140.97 83.82)
 		(diameter 0)
 		(color 0 0 0 0)
@@
 	(wire
 		(pts
-			(xy 102.87 86.36) (xy 140.97 86.36)
+			(xy 102.87 83.82) (xy 140.97 83.82)
+		)
+		(stroke
+			(width 0)
+			(type default)
+		)
+	)
+	(wire
+		(pts
+			(xy 102.87 83.82) (xy 102.87 86.36)
 		)
 		(stroke
@@
 	(wire
 		(pts
-			(xy 186.69 73.66) (xy 186.69 74.93)
-		)
-		(stroke
-			(width 0)
-			(type default)
-		)
-	)
-	(wire
-		(pts
 			(xy 128.27 105.41) (xy 128.27 119.38)
 		)
@@
 	(wire
 		(pts
-			(xy 140.97 78.74) (xy 140.97 86.36)
+			(xy 140.97 78.74) (xy 140.97 83.82)
 		)
 		(stroke
@@
 	(wire
 		(pts
-			(xy 140.97 86.36) (xy 140.97 92.71)
+			(xy 140.97 83.82) (xy 140.97 92.71)
 		)
 		(stroke
@@
 			(width 0)
 			(type default)
+		)
+	)
+	(text "je sais pas si ça marche\nc'est la merde"
+		(exclude_from_sim no)
+		(at 192.786 161.544 0)
+		(effects
+			(font
+				(size 1.27 1.27)
+			)
+		)
+	)
+	(text "chgmt composants en 5,5 V et rajout pont H pour entree"
+		(exclude_from_sim no)
+		(at 166.878 59.944 0)
+		(effects
+			(font
+				(size 1.27 1.27)
+			)
 		)
 	)
 	(hierarchical_label "set"
 		(shape input)
-		(at 97.79 109.22 0)
-		(fields_autoplaced yes)
-		(effects
-			(font
-				(size 1.27 1.27)
-			)
-			(justify left)
+		(at 97.79 109.22 270)
+		(fields_autoplaced yes)
+		(effects
+			(font
+				(size 1.27 1.27)
+			)
+			(justify right)
 		)
 	)
 	(hierarchical_label "set"
 		(shape input)
-		(at 132.08 40.64 0)
+		(at 132.08 40.64 90)
 		(fields_autoplaced yes)
 		(effects
@@
 	(hierarchical_label "230 V sortie"
 		(shape output)
-		(at 186.69 74.93 0)
+		(at 186.69 73.66 0)
 		(fields_autoplaced yes)
 		(effects
@@
 	(hierarchical_label "reset"
 		(shape input)
-		(at 128.27 119.38 0)
-		(fields_autoplaced yes)
-		(effects
-			(font
-				(size 1.27 1.27)
-			)
-			(justify left)
-		)
-	)
+		(at 128.27 119.38 270)
+		(fields_autoplaced yes)
+		(effects
+			(font
+				(size 1.27 1.27)
+			)
+			(justify right)
+		)
+	)

Commit message: Maj schéma
Parts:
- renumbered Q3 to Q1, Q4 to Q2, Q2 to Q3, Q1 to Q4, R25 to R27, R27 to R28, R24 to R29, U5 to U7
Changed lines of the file:
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@@
 		(dnp no)
 		(fields_autoplaced yes)
-		(property "Reference" "R27"
+		(property "Reference" "R28"
 			(at 130.81 101.5999 0)
 			(effects
@@
 		(instances
 			(project "FabOS_MB"
-				(path "/09377d5d-727f-4ff4-92c8-7a0483d23f1e/1adf3e9b-e12c-4a02-81a9-1b622a2960c2"
-					(reference "R27")
+				(path "/09377d5d-727f-4ff4-92c8-7a0483d23f1e/c1d99fe3-76d7-4388-b359-2aa0cf96dce1"
+					(reference "R28")
 					(unit 1)
 				)
@@
 		(on_board yes)
 		(dnp no)
-		(property "Reference" "Q2"
+		(property "Reference" "Q3"
 			(at 128.27 86.36 90)
 			(effects
@@
 		(instances
 			(project "FabOS_MB"
-				(path "/09377d5d-727f-4ff4-92c8-7a0483d23f1e/1adf3e9b-e12c-4a02-81a9-1b622a2960c2"
-					(reference "Q2")
+				(path "/09377d5d-727f-4ff4-92c8-7a0483d23f1e/c1d99fe3-76d7-4388-b359-2aa0cf96dce1"
+					(reference "Q3")
 					(unit 1)
 				)
@@
 		(instances
 			(project "FabOS_MB"
-				(path "/09377d5d-727f-4ff4-92c8-7a0483d23f1e/1adf3e9b-e12c-4a02-81a9-1b622a2960c2"
+				(path "/09377d5d-727f-4ff4-92c8-7a0483d23f1e/c1d99fe3-76d7-4388-b359-2aa0cf96dce1"
 					(reference "R26")
 					(unit 1)
@@
 		(dnp no)
 		(fields_autoplaced yes)
-		(property "Reference" "#PWR023"
+		(property "Reference" "#PWR033"
 			(at 113.03 58.42 0)
 			(effects
@@
 		(instances
 			(project "FabOS_MB"
-				(path "/09377d5d-727f-4ff4-92c8-7a0483d23f1e/1adf3e9b-e12c-4a02-81a9-1b622a2960c2"
-					(reference "#PWR023")
+				(path "/09377d5d-727f-4ff4-92c8-7a0483d23f1e/c1d99fe3-76d7-4388-b359-2aa0cf96dce1"
+					(reference "#PWR033")
 					(unit 1)
 				)
@@
 		(on_board yes)
 		(dnp no)
-		(property "Reference" "Q3"
+		(property "Reference" "Q1"
 			(at 97.79 80.01 90)
 			(effects
@@
 		(instances
 			(project "FabOS_MB"
-				(path "/09377d5d-727f-4ff4-92c8-7a0483d23f1e/1adf3e9b-e12c-4a02-81a9-1b622a2960c2"
-					(reference "Q3")
+				(path "/09377d5d-727f-4ff4-92c8-7a0483d23f1e/c1d99fe3-76d7-4388-b359-2aa0cf96dce1"
+					(reference "Q1")
 					(unit 1)
 				)
@@
 		(dnp no)
 		(fields_autoplaced yes)
-		(property "Reference" "R24"
+		(property "Reference" "R29"
 			(at 134.62 45.7199 0)
 			(effects
@@
 		(instances
 			(project "FabOS_MB"
-				(path "/09377d5d-727f-4ff4-92c8-7a0483d23f1e/1adf3e9b-e12c-4a02-81a9-1b622a2960c2"
-					(reference "R24")
+				(path "/09377d5d-727f-4ff4-92c8-7a0483d23f1e/c1d99fe3-76d7-4388-b359-2aa0cf96dce1"
+					(reference "R29")
 					(unit 1)
 				)
@@
 		(dnp no)
 		(fields_autoplaced yes)
-		(property "Reference" "Q1"
+		(property "Reference" "Q4"
 			(at 132.08 62.23 90)
 			(effects
@@
 		)
 		(instances
-			(project ""
-				(path "/09377d5d-727f-4ff4-92c8-7a0483d23f1e/1adf3e9b-e12c-4a02-81a9-1b622a2960c2"
-					(reference "Q1")
+			(project "FabOS_MB"
+				(path "/09377d5d-727f-4ff4-92c8-7a0483d23f1e/c1d99fe3-76d7-4388-b359-2aa0cf96dce1"
+					(reference "Q4")
 					(unit 1)
 				)
@@
 		(dnp no)
 		(fields_autoplaced yes)
-		(property "Reference" "R25"
+		(property "Reference" "R27"
 			(at 115.57 76.2 90)
 			(effects
@@
 		(instances
 			(project "FabOS_MB"
-				(path "/09377d5d-727f-4ff4-92c8-7a0483d23f1e/1adf3e9b-e12c-4a02-81a9-1b622a2960c2"
-					(reference "R25")
+				(path "/09377d5d-727f-4ff4-92c8-7a0483d23f1e/c1d99fe3-76d7-4388-b359-2aa0cf96dce1"
+					(reference "R27")
 					(unit 1)
 				)
@@
 		(dnp no)
 		(fields_autoplaced yes)
-		(property "Reference" "#PWR024"
+		(property "Reference" "#PWR034"
 			(at 171.45 93.98 0)
 			(effects
@@
 		)
 		(instances
-			(project ""
-				(path "/09377d5d-727f-4ff4-92c8-7a0483d23f1e/1adf3e9b-e12c-4a02-81a9-1b622a2960c2"
-					(reference "#PWR024")
+			(project "FabOS_MB"
+				(path "/09377d5d-727f-4ff4-92c8-7a0483d23f1e/c1d99fe3-76d7-4388-b359-2aa0cf96dce1"
+					(reference "#PWR034")
 					(unit 1)
 				)
@@
 		(on_board yes)
 		(dnp no)
-		(property "Reference" "U5"
+		(property "Reference" "U7"
 			(at 153.035 66.04 0)
 			(effects
@@
 		(instances
 			(project "FabOS_MB"
-				(path "/09377d5d-727f-4ff4-92c8-7a0483d23f1e/1adf3e9b-e12c-4a02-81a9-1b622a2960c2"
-					(reference "U5")
+				(path "/09377d5d-727f-4ff4-92c8-7a0483d23f1e/c1d99fe3-76d7-4388-b359-2aa0cf96dce1"
+					(reference "U7")
 					(unit 1)
 				)
@@
 		(dnp no)
 		(fields_autoplaced yes)
-		(property "Reference" "#PWR022"
+		(property "Reference" "#PWR032"
 			(at 109.22 92.71 0)
 			(effects
@@
 		)
 		(instances
-			(project ""
-				(path "/09377d5d-727f-4ff4-92c8-7a0483d23f1e/1adf3e9b-e12c-4a02-81a9-1b622a2960c2"
-					(reference "#PWR022")
+			(project "FabOS_MB"
+				(path "/09377d5d-727f-4ff4-92c8-7a0483d23f1e/c1d99fe3-76d7-4388-b359-2aa0cf96dce1"
+					(reference "#PWR032")
 					(unit 1)
 				)
@@
 		(on_board yes)
 		(dnp no)
-		(property "Reference" "Q4"
+		(property "Reference" "Q2"
 			(at 123.19 67.31 90)
 			(effects
@@
 		(instances
 			(project "FabOS_MB"
-				(path "/09377d5d-727f-4ff4-92c8-7a0483d23f1e/1adf3e9b-e12c-4a02-81a9-1b622a2960c2"
-					(reference "Q4")
-					(unit 1)
-				)
+				(path "/09377d5d-727f-4ff4-92c8-7a0483d23f1e/c1d99fe3-76d7-4388-b359-2aa0cf96dce1"
+					(reference "Q2")
+					(unit 1)
+				)

Commit message: ajout nom des composants pour 5v
Parts:
- removed Q1, Q2, Q3, Q4: NMOS, symbol Simulation_SPICE:NMOS
- removed R26, R27, R28, R29: 22, Resistor_SMD:R_0402_1005Metric, symbol Device:R_Small
Connections:
- net 230 V entrée: no longer names the net of U7.L (Vin)
Other:
- note added: "chgmt composants en 5,5 V et rajout pont H pour entree Omron Electronics G6KU-2F-Y-TR DC5 https://www.lcsc.com/product-detail/Magnetic-Latching-Relays_Omron-Electronics-G6KU-2F-Y-TR-DC5_C2153173.html Texas Instruments DRV8220DRLR https://www.ti.com/lit/ds/symlink/drv8220.pdf?ts=1718862780189&ref_url=https%253A%252F%252Fwww.ti.com%252Fproduct%252FDRV8220%253Futm_source%253Dgoogle%2526utm_medium%25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"
- note removed: "chgmt composants en 5,5 V et rajout pont H pour entree"
- note removed: "je sais pas si ça marche c'est la merde"
- moved on the sheet: U7

Commit message: comopsants switch et ethernets fini?
Parts:
- removed U7: HF3F-L 12-1ZL1T, Librairie_MB:switch 12V, symbol Librairie_MB:Switch_12V
- added C20: Cbulk, symbol Device:C_Small
- added C22: 0,1µ, symbol Device:C_Small
- added U10: ~, Librairie_MB:relay driver, symbol Librairie_MB:relay_driver
- added U7: ~, Librairie_MB:switch 5V, symbol Librairie_MB:switch_5V
Connections:
- net 230 V sortie: now also U7.6 (L_output)
- new net: U10.4 (OUT2), U7.1 (set_+)
- new net: U10.6 (OUT1), U7.8 (reset_+)
- new net 12V: C20.2, C22.2, U10.5 (VM)
- new net Ctrl1: U10.1 (IN1)
- new net Ctrl2: U10.2 (IN2)
- new net GND: C20.1, C22.1, U10.3 (GND)
- new net L input: U7.7 (L)
- no-connect marks 0 -> 4
Other:
- note removed: "chgmt composants en 5,5 V et rajout pont H pour entree Omron Electronics G6KU-2F-Y-TR DC5 https://www.lcsc.com/product-detail/Magnetic-Latching-Relays_Omron-Electronics-G6KU-2F-Y-TR-DC5_C2153173.html Texas Instruments DRV8220DRLR https://www.ti.com/lit/ds/symlink/drv8220.pdf?ts=1718862780189&ref_url=https%253A%252F%252Fwww.ti.com%252Fproduct%252FDRV8220%253Futm_source%253Dgoogle%2526utm_medium%25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"
