File: FabOS_MB/pouissance.kicad_sch (KiCad schematic)
At the start: 13 parts, among them U2 TPS563201, U6 TDPOWER TAS10-12-W2

Commit message: Schéma LIN
Je n'ai pas compris comment l'alim fonctionne
Other:
- moved on the sheet: C1, C2, C3, C4, C7, C8, C9, L1, R1, R2, R5, U2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

Commit message: Maj schéma
Parts:
- renumbered C9 to C1, C8 to C2, C1 to C3, C2 to C4, C3 to C5, C7 to C6, C4 to C7, R5 to R1, R1 to R3, U6 to U3
Changed lines of the file:
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@@
 		(dnp no)
 		(fields_autoplaced yes)
-		(property "Reference" "R5"
+		(property "Reference" "R1"
 			(at 146.05 91.44 90)
 			(effects
@@
 		)
 		(instances
-			(project ""
-				(path "/09377d5d-727f-4ff4-92c8-7a0483d23f1e/551154e0-2135-4b34-9e32-981e3d52220b"
-					(reference "R5")
+			(project "FabOS_MB"
+				(path "/09377d5d-727f-4ff4-92c8-7a0483d23f1e/e6afd72f-9acd-432b-896e-1ebfe08116f3"
+					(reference "R1")
 					(unit 1)
 				)
@@
 		(dnp no)
 		(fields_autoplaced yes)
-		(property "Reference" "U6"
+		(property "Reference" "U3"
 			(at 231.14 86.36 0)
 			(effects
@@
 		(instances
 			(project "FabOS_MB"
-				(path "/09377d5d-727f-4ff4-92c8-7a0483d23f1e/551154e0-2135-4b34-9e32-981e3d52220b"
-					(reference "U6")
+				(path "/09377d5d-727f-4ff4-92c8-7a0483d23f1e/e6afd72f-9acd-432b-896e-1ebfe08116f3"
+					(reference "U3")
 					(unit 1)
 				)
@@
 		(dnp no)
 		(fields_autoplaced yes)
-		(property "Reference" "C4"
+		(property "Reference" "C7"
 			(at 179.0763 106.68 90)
 			(effects
@@
 		)
 		(instances
-			(project ""
-				(path "/09377d5d-727f-4ff4-92c8-7a0483d23f1e/551154e0-2135-4b34-9e32-981e3d52220b"
-					(reference "C4")
+			(project "FabOS_MB"
+				(path "/09377d5d-727f-4ff4-92c8-7a0483d23f1e/e6afd72f-9acd-432b-896e-1ebfe08116f3"
+					(reference "C7")
 					(unit 1)
 				)
@@
 		(dnp no)
 		(fields_autoplaced yes)
-		(property "Reference" "C7"
+		(property "Reference" "C6"
 			(at 128.2763 71.12 90)
 			(effects
@@
 		)
 		(instances
-			(project ""
-				(path "/09377d5d-727f-4ff4-92c8-7a0483d23f1e/551154e0-2135-4b34-9e32-981e3d52220b"
-					(reference "C7")
+			(project "FabOS_MB"
+				(path "/09377d5d-727f-4ff4-92c8-7a0483d23f1e/e6afd72f-9acd-432b-896e-1ebfe08116f3"
+					(reference "C6")
 					(unit 1)
 				)
@@
 		(instances
 			(project "FabOS_MB"
-				(path "/09377d5d-727f-4ff4-92c8-7a0483d23f1e/551154e0-2135-4b34-9e32-981e3d52220b"
+				(path "/09377d5d-727f-4ff4-92c8-7a0483d23f1e/e6afd72f-9acd-432b-896e-1ebfe08116f3"
 					(reference "U2")
 					(unit 1)
@@
 		(dnp no)
 		(fields_autoplaced yes)
-		(property "Reference" "#PWR07"
+		(property "Reference" "#PWR014"
 			(at 156.21 119.38 0)
 			(effects
@@
 		)
 		(instances
-			(project ""
-				(path "/09377d5d-727f-4ff4-92c8-7a0483d23f1e/551154e0-2135-4b34-9e32-981e3d52220b"
-					(reference "#PWR07")
+			(project "FabOS_MB"
+				(path "/09377d5d-727f-4ff4-92c8-7a0483d23f1e/e6afd72f-9acd-432b-896e-1ebfe08116f3"
+					(reference "#PWR014")
 					(unit 1)
 				)
@@
 		(dnp no)
 		(fields_autoplaced yes)
-		(property "Reference" "C2"
+		(property "Reference" "C4"
 			(at 80.01 101.6062 0)
 			(effects
@@
 		)
 		(instances
-			(project ""
-				(path "/09377d5d-727f-4ff4-92c8-7a0483d23f1e/551154e0-2135-4b34-9e32-981e3d52220b"
-					(reference "C2")
+			(project "FabOS_MB"
+				(path "/09377d5d-727f-4ff4-92c8-7a0483d23f1e/e6afd72f-9acd-432b-896e-1ebfe08116f3"
+					(reference "C4")
 					(unit 1)
 				)
@@
 		(dnp no)
 		(fields_autoplaced yes)
-		(property "Reference" "C1"
+		(property "Reference" "C3"
 			(at 67.31 101.6062 0)
 			(effects
@@
 		)
 		(instances
-			(project ""
-				(path "/09377d5d-727f-4ff4-92c8-7a0483d23f1e/551154e0-2135-4b34-9e32-981e3d52220b"
-					(reference "C1")
+			(project "FabOS_MB"
+				(path "/09377d5d-727f-4ff4-92c8-7a0483d23f1e/e6afd72f-9acd-432b-896e-1ebfe08116f3"
+					(reference "C3")
 					(unit 1)
 				)
@@
 		(dnp no)
 		(fields_autoplaced yes)
-		(property "Reference" "R1"
+		(property "Reference" "R3"
 			(at 179.07 96.52 90)
 			(effects
@@
 		)
 		(instances
-			(project ""
-				(path "/09377d5d-727f-4ff4-92c8-7a0483d23f1e/551154e0-2135-4b34-9e32-981e3d52220b"
-					(reference "R1")
+			(project "FabOS_MB"
+				(path "/09377d5d-727f-4ff4-92c8-7a0483d23f1e/e6afd72f-9acd-432b-896e-1ebfe08116f3"
+					(reference "R3")
 					(unit 1)
 				)
@@
 		(dnp no)
 		(fields_autoplaced yes)
-		(property "Reference" "#PWR05"
+		(property "Reference" "#PWR013"
 			(at 110.49 90.17 0)
 			(effects
@@
 		)
 		(instances
-			(project ""
-				(path "/09377d5d-727f-4ff4-92c8-7a0483d23f1e/551154e0-2135-4b34-9e32-981e3d52220b"
-					(reference "#PWR05")
+			(project "FabOS_MB"
+				(path "/09377d5d-727f-4ff4-92c8-7a0483d23f1e/e6afd72f-9acd-432b-896e-1ebfe08116f3"
+					(reference "#PWR013")
 					(unit 1)
 				)
@@
 		(dnp no)
 		(fields_autoplaced yes)
-		(property "Reference" "#PWR06"
+		(property "Reference" "#PWR012"
 			(at 52.07 100.33 0)
 			(effects
@@
 		)
 		(instances
-			(project ""
-				(path "/09377d5d-727f-4ff4-92c8-7a0483d23f1e/551154e0-2135-4b34-9e32-981e3d52220b"
-					(reference "#PWR06")
+			(project "FabOS_MB"
+				(path "/09377d5d-727f-4ff4-92c8-7a0483d23f1e/e6afd72f-9acd-432b-896e-1ebfe08116f3"
+					(reference "#PWR012")
 					(unit 1)
 				)
@@
 		)
 		(instances
-			(project ""
-				(path "/09377d5d-727f-4ff4-92c8-7a0483d23f1e/551154e0-2135-4b34-9e32-981e3d52220b"
+			(project "FabOS_MB"
+				(path "/09377d5d-727f-4ff4-92c8-7a0483d23f1e/e6afd72f-9acd-432b-896e-1ebfe08116f3"
 					(reference "L1")
 					(unit 1)
@@
 		(dnp no)
 		(fields_autoplaced yes)
-		(property "Reference" "C8"
+		(property "Reference" "C2"
 			(at 60.96 91.4462 0)
 			(effects
@@
 		)
 		(instances
-			(project ""
-				(path "/09377d5d-727f-4ff4-92c8-7a0483d23f1e/551154e0-2135-4b34-9e32-981e3d52220b"
-					(reference "C8")
+			(project "FabOS_MB"
+				(path "/09377d5d-727f-4ff4-92c8-7a0483d23f1e/e6afd72f-9acd-432b-896e-1ebfe08116f3"
+					(reference "C2")
 					(unit 1)
 				)
@@
 		(dnp no)
 		(fields_autoplaced yes)
-		(property "Reference" "C9"
+		(property "Reference" "C1"
 			(at 46.99 91.4462 0)
 			(effects
@@
 		)
 		(instances
-			(project ""
-				(path "/09377d5d-727f-4ff4-92c8-7a0483d23f1e/551154e0-2135-4b34-9e32-981e3d52220b"
-					(reference "C9")
+			(project "FabOS_MB"
+				(path "/09377d5d-727f-4ff4-92c8-7a0483d23f1e/e6afd72f-9acd-432b-896e-1ebfe08116f3"
+					(reference "C1")
 					(unit 1)
 				)
@@
 		)
 		(instances
-			(project ""
-				(path "/09377d5d-727f-4ff4-92c8-7a0483d23f1e/551154e0-2135-4b34-9e32-981e3d52220b"
+			(project "FabOS_MB"
+				(path "/09377d5d-727f-4ff4-92c8-7a0483d23f1e/e6afd72f-9acd-432b-896e-1ebfe08116f3"
 					(reference "R2")
 					(unit 1)
@@
 		(dnp no)
 		(fields_autoplaced yes)
-		(property "Reference" "C3"
+		(property "Reference" "C5"
 			(at 93.98 101.6062 0)
 			(effects
@@
 		)
 		(instances
-			(project ""
-				(path "/09377d5d-727f-4ff4-92c8-7a0483d23f1e/551154e0-2135-4b34-9e32-981e3d52220b"
-					(reference "C3")
+			(project "FabOS_MB"
+				(path "/09377d5d-727f-4ff4-92c8-7a0483d23f1e/e6afd72f-9acd-432b-896e-1ebfe08116f3"
+					(reference "C5")
 					(unit 1)
 				)
@@
 		(dnp no)
 		(fields_autoplaced yes)
-		(property "Reference" "#PWR04"
+		(property "Reference" "#PWR015"
 			(at 246.38 100.33 0)
 			(effects
@@
 		)
 		(instances
-			(project ""
-				(path "/09377d5d-727f-4ff4-92c8-7a0483d23f1e/551154e0-2135-4b34-9e32-981e3d52220b"
-					(reference "#PWR04")
-					(unit 1)
-				)
+			(project "FabOS_MB"
+				(path "/09377d5d-727f-4ff4-92c8-7a0483d23f1e/e6afd72f-9acd-432b-896e-1ebfe08116f3"
+					(reference "#PWR015")
+					(unit 1)
+				)

Commit message: Maj 5V
Parts:
- C1, C2: value 22µ -> 22u
- L1: value 2,2µ -> 2,2u
- U3: value TDPOWER TAS10-12-W2 -> TDPOWER TAS12-5-W2; LCSC C2687656 -> C5354760; MPN TAS10-12-W2 -> TAS12-5-W2
Connections:
- net 12V renamed 5V
Changed lines of the file:
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@@
 	(wire
 		(pts
-			(xy 250.19 104.14) (xy 246.38 104.14)
+			(xy 246.38 104.14) (xy 247.65 104.14)
 		)
 		(stroke
@@
 	(wire
 		(pts
-			(xy 251.46 107.95) (xy 250.19 107.95)
-		)
-		(stroke
-			(width 0)
-			(type default)
-		)
-	)
-	(wire
-		(pts
 			(xy 142.24 90.17) (xy 149.86 90.17)
 		)
@@
 	(wire
 		(pts
-			(xy 250.19 107.95) (xy 250.19 104.14)
-		)
-		(stroke
-			(width 0)
-			(type default)
-		)
-	)
-	(wire
-		(pts
 			(xy 190.5 102.87) (xy 190.5 113.03)
 		)
@@
 		)
 	)
-	(label "V_in"
-		(at 45.72 104.14 180)
+	(hierarchical_label "3V3"
+		(shape output)
+		(at 34.29 90.17 180)
 		(fields_autoplaced yes)
 		(effects
@@
 				(size 1.27 1.27)
 			)
-			(justify right bottom)
-		)
-	)
-	(label "V_in"
-		(at 250.19 104.14 0)
+			(justify right)
+		)
+	)
+	(hierarchical_label "Neutre"
+		(shape input)
+		(at 215.9 104.14 180)
 		(fields_autoplaced yes)
 		(effects
@@
 				(size 1.27 1.27)
 			)
-			(justify left bottom)
-		)
-	)
-	(hierarchical_label "3V3"
-		(shape output)
-		(at 34.29 90.17 180)
+			(justify right)
+		)
+	)
+	(hierarchical_label "EN"
+		(shape input)
+		(at 149.86 97.79 0)
 		(fields_autoplaced yes)
 		(effects
@@
 				(size 1.27 1.27)
 			)
-			(justify right)
-		)
-	)
-	(hierarchical_label "Neutre"
-		(shape input)
-		(at 215.9 104.14 180)
+			(justify left)
+		)
+	)
+	(hierarchical_label "5V"
+		(shape output)
+		(at 247.65 104.14 0)
 		(fields_autoplaced yes)
 		(effects
@@
 				(size 1.27 1.27)
 			)
-			(justify right)
-		)
-	)
-	(hierarchical_label "EN"
+			(justify left)
+		)
+	)
+	(hierarchical_label "3V3"
 		(shape input)
-		(at 149.86 97.79 0)
+		(at 190.5 102.87 0)
 		(fields_autoplaced yes)
 		(effects
@@
 		)
 	)
-	(hierarchical_label "12V"
-		(shape output)
-		(at 251.46 107.95 0)
+	(hierarchical_label "5V"
+		(shape input)
+		(at 45.72 104.14 180)
 		(fields_autoplaced yes)
 		(effects
@@
 				(size 1.27 1.27)
 			)
-			(justify left)
-		)
-	)
-	(hierarchical_label "3V3"
-		(shape input)
-		(at 190.5 102.87 0)
-		(fields_autoplaced yes)
-		(effects
-			(font
-				(size 1.27 1.27)
-			)
-			(justify left)
+			(justify right)
 		)
 	)
@@
 			)
 		)
-		(property "Value" "TDPOWER TAS10-12-W2"
+		(property "Value" "TDPOWER TAS12-5-W2"
 			(at 231.14 88.9 0)
 			(effects
@@
 			)
 		)
-		(property "Datasheet" "https://www.lcsc.com/datasheet/lcsc_datasheet_2109141830_TDPOWER-TAS10-12-W2_C2687656.pdf"
+		(property "Datasheet" "https://www.lcsc.com/datasheet/lcsc_datasheet_2307141637_TDPOWER-TAS12-5-W2_C5354760.pdf"
 			(at 231.14 99.06 0)
 			(effects
@@
 			)
 		)
-		(property "MPN" "TAS10-12-W2"
+		(property "MPN" "TAS12-5-W2"
 			(at 231.14 99.06 0)
 			(effects
@@
 			)
 		)
-		(property "LCSC" " C2687656"
+		(property "LCSC" "C5354760"
 			(at 231.14 99.06 0)
 			(effects
@@
 			)
 		)
-		(property "Value" "2,2µ"
+		(property "Value" "2,2u"
 			(at 82.55 87.63 90)
 			(effects
@@
 			)
 		)
-		(property "Value" "22µ"
+		(property "Value" "22u"
 			(at 60.96 93.9862 0)
 			(effects
@@
 			)
 		)
-		(property "Value" "22µ"
+		(property "Value" "22u"
 			(at 46.99 93.9862 0)
 			(effects

Commit message: Schéma processeur
Parts:
- C3, C4: value C_Small -> 10u; Matériau (none) -> Céramique
- C5, C6: value C_Small -> 100n
- R1: value R -> 10k
Changed lines of the file:
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@@
 			)
 		)
-		(property "Value" "R"
+		(property "Value" "10k"
 			(at 146.05 93.98 90)
 			(effects
@@
 			)
 		)
-		(property "Value" "C_Small"
+		(property "Value" "100n"
 			(at 128.2763 73.66 90)
 			(effects
@@
 		(on_board yes)
 		(dnp no)
-		(fields_autoplaced yes)
 		(property "Reference" "C4"
 			(at 80.01 101.6062 0)
@@
 			)
 		)
-		(property "Value" "C_Small"
+		(property "Value" "10u"
 			(at 80.01 104.1462 0)
 			(effects
@@
 			)
 		)
+		(property "Matériau" "Céramique"
+			(at 77.47 107.442 0)
+			(effects
+				(font
+					(size 1.27 1.27)
+				)
+			)
+		)
 		(pin "2"
 		)
@@
 		(on_board yes)
 		(dnp no)
-		(fields_autoplaced yes)
 		(property "Reference" "C3"
 			(at 67.31 101.6062 0)
@@
 			)
 		)
-		(property "Value" "C_Small"
+		(property "Value" "10u"
 			(at 67.31 104.1462 0)
 			(effects
@@
 			)
 		)
+		(property "Matériau" "Céramique"
+			(at 64.77 107.188 0)
+			(effects
+				(font
+					(size 1.27 1.27)
+				)
+			)
+		)
 		(pin "1"
 		)
@@
 			)
 		)
-		(property "Value" "C_Small"
+		(property "Value" "100n"
 			(at 93.98 104.1462 0)
 			(effects

Commit message: Correction de certaines erreurs
Parts:
- renumbered U2 to U1, U3 to U2
Changed lines of the file:
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@@
+		)
+	)
+	(label "3.3V"
+		(at 190.5 102.87 0)
+		(fields_autoplaced yes)
+		(effects
+			(font
+				(size 1.27 1.27)
+			)
+			(justify left bottom)
+		)
+	)
+	(label "3.3V"
+		(at 44.45 90.17 0)
+		(fields_autoplaced yes)
+		(effects
+			(font
+				(size 1.27 1.27)
+			)
+			(justify left bottom)
 		)
 	)
@@
 		)
 	)
-	(hierarchical_label "3V3"
+	(hierarchical_label "5V"
 		(shape input)
-		(at 190.5 102.87 0)
+		(at 45.72 104.14 180)
 		(fields_autoplaced yes)
 		(effects
@@
 				(size 1.27 1.27)
 			)
-			(justify left)
-		)
-	)
-	(hierarchical_label "5V"
+			(justify right)
+		)
+	)
+	(hierarchical_label "Phase"
 		(shape input)
-		(at 45.72 104.14 180)
+		(at 215.9 93.98 180)
 		(fields_autoplaced yes)
 		(effects
@@
 		)
 	)
-	(hierarchical_label "Phase"
-		(shape input)
-		(at 215.9 93.98 180)
-		(fields_autoplaced yes)
-		(effects
-			(font
-				(size 1.27 1.27)
-			)
-			(justify right)
-		)
-	)
 	(symbol
 		(lib_id "Device:R")
@@
 		(dnp no)
 		(fields_autoplaced yes)
-		(property "Reference" "U3"
+		(property "Reference" "U2"
 			(at 231.14 86.36 0)
 			(effects
@@
 			(project "FabOS_MB"
 				(path "/09377d5d-727f-4ff4-92c8-7a0483d23f1e/e6afd72f-9acd-432b-896e-1ebfe08116f3"
-					(reference "U3")
+					(reference "U2")
 					(unit 1)
 				)
@@
 		(on_board yes)
 		(dnp no)
-		(property "Reference" "U2"
+		(property "Reference" "U1"
 			(at 129.8575 83.82 0)
 			(effects
@@
 			(project "FabOS_MB"
 				(path "/09377d5d-727f-4ff4-92c8-7a0483d23f1e/e6afd72f-9acd-432b-896e-1ebfe08116f3"
-					(reference "U2")
+					(reference "U1")
 					(unit 1)
 				)
@@
 		(dnp no)
 		(fields_autoplaced yes)
-		(property "Reference" "#PWR014"
+		(property "Reference" "#PWR017"
 			(at 156.21 119.38 0)
 			(effects
@@
 			(project "FabOS_MB"
 				(path "/09377d5d-727f-4ff4-92c8-7a0483d23f1e/e6afd72f-9acd-432b-896e-1ebfe08116f3"
-					(reference "#PWR014")
+					(reference "#PWR017")
 					(unit 1)
 				)
@@
 		(dnp no)
 		(fields_autoplaced yes)
-		(property "Reference" "#PWR013"
+		(property "Reference" "#PWR016"
 			(at 110.49 90.17 0)
 			(effects
@@
 			(project "FabOS_MB"
 				(path "/09377d5d-727f-4ff4-92c8-7a0483d23f1e/e6afd72f-9acd-432b-896e-1ebfe08116f3"
-					(reference "#PWR013")
+					(reference "#PWR016")
 					(unit 1)
 				)
@@
 		(dnp no)
 		(fields_autoplaced yes)
-		(property "Reference" "#PWR012"
+		(property "Reference" "#PWR015"
 			(at 52.07 100.33 0)
 			(effects
@@
 			(project "FabOS_MB"
 				(path "/09377d5d-727f-4ff4-92c8-7a0483d23f1e/e6afd72f-9acd-432b-896e-1ebfe08116f3"
-					(reference "#PWR012")
+					(reference "#PWR015")
 					(unit 1)
 				)
@@
 		(dnp no)
 		(fields_autoplaced yes)
-		(property "Reference" "#PWR015"
+		(property "Reference" "#PWR018"
 			(at 246.38 100.33 0)
 			(effects
@@
 			(project "FabOS_MB"
 				(path "/09377d5d-727f-4ff4-92c8-7a0483d23f1e/e6afd72f-9acd-432b-896e-1ebfe08116f3"
-					(reference "#PWR015")
-					(unit 1)
-				)
+					(reference "#PWR018")
+					(unit 1)
+				)

Commit message: petits test de correction
Connections:
- net 3V3 renamed +3.3V
Changed lines of the file:
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@@
 		)
 	)
-	(label "3.3V"
+	(global_label "+3.3V"
+		(shape input)
 		(at 190.5 102.87 0)
 		(fields_autoplaced yes)
@@
 				(size 1.27 1.27)
 			)
-			(justify left bottom)
+			(justify left)
+		)
+		(property "Intersheetrefs" "${INTERSHEET_REFS}"
+			(at 199.17 102.87 0)
+			(effects
+				(font
+					(size 1.27 1.27)
+				)
+				(justify left)
+				(hide yes)
+			)
 		)
 	)
-	(label "3.3V"
-		(at 44.45 90.17 0)
-		(fields_autoplaced yes)
-		(effects
-			(font
-				(size 1.27 1.27)
-			)
-			(justify left bottom)
-		)
-	)
-	(hierarchical_label "3V3"
+	(global_label "+3.3V"
 		(shape output)
 		(at 34.29 90.17 180)
@@
 			(justify right)
 		)
+		(property "Intersheetrefs" "${INTERSHEET_REFS}"
+			(at 25.62 90.17 0)
+			(effects
+				(font
+					(size 1.27 1.27)
+				)
+				(justify right)
+				(hide yes)
+			)
+		)
 	)

Commit message: Il ne reste plus qu'a router
Parts:
- removed C7: C_Small, symbol Device:C_Small
Connections:
- net +3.3V: no longer R3.2
Changed lines of the file:
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@@
-	)
-	(junction
-		(at 166.37 105.41)
-		(diameter 0)
-		(color 0 0 0 0)
 	)
 	(junction
@@
 	(wire
 		(pts
-			(xy 190.5 113.03) (xy 181.61 113.03)
-		)
-		(stroke
-			(width 0)
-			(type default)
-		)
-	)
-	(wire
-		(pts
 			(xy 64.77 105.41) (xy 77.47 105.41)
 		)
@@
 	(wire
 		(pts
-			(xy 166.37 113.03) (xy 166.37 105.41)
-		)
-		(stroke
-			(width 0)
-			(type default)
-		)
-	)
-	(wire
-		(pts
 			(xy 44.45 95.25) (xy 58.42 95.25)
 		)
@@
 	(wire
 		(pts
-			(xy 176.53 113.03) (xy 166.37 113.03)
-		)
-		(stroke
-			(width 0)
-			(type default)
-		)
-	)
-	(wire
-		(pts
-			(xy 190.5 102.87) (xy 190.5 113.03)
-		)
-		(stroke
-			(width 0)
-			(type default)
-		)
-	)
-	(wire
-		(pts
 			(xy 182.88 102.87) (xy 190.5 102.87)
 		)
@@
 			(width 0)
 			(type default)
-		)
-	)
-	(global_label "+3.3V"
-		(shape input)
-		(at 190.5 102.87 0)
-		(fields_autoplaced yes)
-		(effects
-			(font
-				(size 1.27 1.27)
-			)
-			(justify left)
-		)
-		(property "Intersheetrefs" "${INTERSHEET_REFS}"
-			(at 199.17 102.87 0)
-			(effects
-				(font
-					(size 1.27 1.27)
-				)
-				(justify left)
-				(hide yes)
-			)
-		)
-	)
-	(global_label "+3.3V"
-		(shape output)
-		(at 34.29 90.17 180)
-		(fields_autoplaced yes)
-		(effects
-			(font
-				(size 1.27 1.27)
-			)
-			(justify right)
-		)
-		(property "Intersheetrefs" "${INTERSHEET_REFS}"
-			(at 25.62 90.17 0)
-			(effects
-				(font
-					(size 1.27 1.27)
-				)
-				(justify right)
-				(hide yes)
-			)
 		)
 	)
@@
 				(path "/09377d5d-727f-4ff4-92c8-7a0483d23f1e/e6afd72f-9acd-432b-896e-1ebfe08116f3"
 					(reference "U2")
-					(unit 1)
-				)
-			)
-		)
-	)
-	(symbol
-		(lib_id "Device:C_Small")
-		(at 179.07 113.03 90)
-		(unit 1)
-		(exclude_from_sim no)
-		(in_bom yes)
-		(on_board yes)
-		(dnp no)
-		(fields_autoplaced yes)
-		(property "Reference" "C7"
-			(at 179.0763 106.68 90)
-			(effects
-				(font
-					(size 1.27 1.27)
-				)
-			)
-		)
-		(property "Value" "C_Small"
-			(at 179.0763 109.22 90)
-			(effects
-				(font
-					(size 1.27 1.27)
-				)
-			)
-		)
-		(property "Footprint" ""
-			(at 179.07 113.03 0)
-			(effects
-				(font
-					(size 1.27 1.27)
-				)
-				(hide yes)
-			)
-		)
-		(property "Datasheet" "~"
-			(at 179.07 113.03 0)
-			(effects
-				(font
-					(size 1.27 1.27)
-				)
-				(hide yes)
-			)
-		)
-		(property "Description" "Unpolarized capacitor, small symbol"
-			(at 179.07 113.03 0)
-			(effects
-				(font
-					(size 1.27 1.27)
-				)
-				(hide yes)
-			)
-		)
-		(pin "2"
-		)
-		(pin "1"
-		)
-		(instances
-			(project "FabOS_MB"
-				(path "/09377d5d-727f-4ff4-92c8-7a0483d23f1e/e6afd72f-9acd-432b-896e-1ebfe08116f3"
-					(reference "C7")
 					(unit 1)
 				)
@@
 	)
 	(symbol
+		(lib_name "+3.3V_1")
+		(lib_id "power:+3.3V")
+		(at 190.5 102.87 0)
+		(unit 1)
+		(exclude_from_sim no)
+		(in_bom yes)
+		(on_board yes)
+		(dnp no)
+		(fields_autoplaced yes)
+		(property "Reference" "#PWR07"
+			(at 190.5 106.68 0)
+			(effects
+				(font
+					(size 1.27 1.27)
+				)
+				(hide yes)
+			)
+		)
+		(property "Value" "+3.3V"
+			(at 190.5 97.79 0)
+			(effects
+				(font
+					(size 1.27 1.27)
+				)
+			)
+		)
+		(property "Footprint" ""
+			(at 190.5 102.87 0)
+			(effects
+				(font
+					(size 1.27 1.27)
+				)
+				(hide yes)
+			)
+		)
+		(property "Datasheet" ""
+			(at 190.5 102.87 0)
+			(effects
+				(font
+					(size 1.27 1.27)
+				)
+				(hide yes)
+			)
+		)
+		(property "Description" "Power symbol creates a global label with name \"+3.3V\""
+			(at 190.5 102.87 0)
+			(effects
+				(font
+					(size 1.27 1.27)
+				)
+				(hide yes)
+			)
+		)
+		(pin "1"
+		)
+		(instances
+			(project "FabOS_MB"
+				(path "/09377d5d-727f-4ff4-92c8-7a0483d23f1e/e6afd72f-9acd-432b-896e-1ebfe08116f3"
+					(reference "#PWR07")
+					(unit 1)
+				)
+			)
+		)
+	)
+	(symbol
 		(lib_id "Device:R")
 		(at 179.07 102.87 90)
@@
 					(unit 1)
 				)
+			)
+		)
+	)
+	(symbol
+		(lib_id "power:+3.3V")
+		(at 34.29 90.17 0)
+		(unit 1)
+		(exclude_from_sim no)
+		(in_bom yes)
+		(on_board yes)
+		(dnp no)
+		(fields_autoplaced yes)
+		(property "Reference" "#PWR06"
+			(at 34.29 93.98 0)
+			(effects
+				(font
+					(size 1.27 1.27)
+				)
+				(hide yes)
+			)
+		)
+		(property "Value" "+3.3V"
+			(at 34.29 85.09 0)
+			(effects
+				(font
+					(size 1.27 1.27)
+				)
+			)
+		)
+		(property "Footprint" ""
+			(at 34.29 90.17 0)
+			(effects
+				(font
+					(size 1.27 1.27)
+				)
+				(hide yes)
+			)
+		)
+		(property "Datasheet" ""
+			(at 34.29 90.17 0)
+			(effects
+				(font
+					(size 1.27 1.27)
+				)
+				(hide yes)
+			)
+		)
+		(property "Description" "Power symbol creates a global label with name \"+3.3V\""
+			(at 34.29 90.17 0)
+			(effects
+				(font
+					(size 1.27 1.27)
+				)
+				(hide yes)
+			)
+		)
+		(pin "1"
+		)
+		(instances
+			(project "FabOS_MB"
+				(path "/09377d5d-727f-4ff4-92c8-7a0483d23f1e/e6afd72f-9acd-432b-896e-1ebfe08116f3"
+					(reference "#PWR06")
+					(unit 1)
+				)
