File: FabOS_MB/STM32.kicad_sch (KiCad schematic)
At the start: 26 parts, among them SW1 boot, SW3 SW_Push, U1 STM32F407VETx

Commit message: Correction de certaines erreurs
Parts:
- removed C24, C25, C26, C27, C28, C29, C30, C31, C32: 100n, symbol Device:C_Small
- renumbered C42 to C21, C20 to C22, C41 to C23, C22 to C25, C23 to C26, C40 to C27, C33 to C29, C34 to C31, C35 to C33, C36 to C35, C38 to C39, C39 to C41, R26 to R32, SW3 to SW2, U1 to U8
Other:
- moved on the sheet: C27, SW2

Commit message: update pcb
Parts:
- added C601: 100n, symbol Device:C_Small
- C21, C23: value 2.2u -> 2u2
- C41: value 4,7u -> 4u7
Connections:
- net +3.3V: now also U8.6 (VBAT), C601.1
- net GND: now also C601.2
- no-connect marks 70 -> 69
Other:
- note added: "A rajouter : Sonde de programmation (avec uart) 3 boutons user (avec le filtre anti rebond) 3 leds user Sortie un GPIO d'emergency stop pour le faire passer dans le cable avec le LIN"
- note added: "VDD Filtering"
- note added: "VDDA Filtering"
- note added: "VRef Filtering"
- moved on the sheet: C22, C31, C33, C35, C37, C39, C41, R32, SW1
