File: FabOS_MB/lin.kicad_sch (KiCad schematic)
At the start: 2 parts, among them J1 USB_A, U3 NCV7329

Commit message: Schéma LIN
Je n'ai pas compris comment l'alim fonctionne
Parts:
- added C13: 10µ, symbol Device:C_Small
- added C14: 220µ, symbol Device:C_Small
- added R23: 10k, symbol Device:R
Connections:
- net 12V: now reaches J1.1 (VBUS)
- net 12V: now also C13.1, R23.1
- net LIN: now reaches J1.2 (D-)
- net LIN: now also J1.3 (D+), U3.6 (LIN), C14.1
- net GND: now reaches J1.4 (GND)
- net GND: now also U3.5 (GND), C13.2, C14.2
- net RXD: now reaches U3.1 (RxD)
- net RXD: now also R23.2
- net EN: now reaches U3.2 (EN)
Other:
- note added: "Pour l'alimentation du LIN je n'ai pas compris la doc"
- moved on the sheet: J1, U3

Commit message: Maj schéma
Parts:
- renumbered C13 to C20, C14 to C21, J1 to J3, R23 to R32, U3 to U9
Changed lines of the file:
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@@
 		(dnp no)
 		(fields_autoplaced yes)
-		(property "Reference" "C13"
+		(property "Reference" "C20"
 			(at 186.69 77.4762 0)
 			(effects
@@
 		)
 		(instances
-			(project ""
-				(path "/09377d5d-727f-4ff4-92c8-7a0483d23f1e/b17da045-52ee-4779-bbc6-bef1d0f1615b"
-					(reference "C13")
+			(project "FabOS_MB"
+				(path "/09377d5d-727f-4ff4-92c8-7a0483d23f1e/0151d859-0a6d-4dae-80c2-9bd1219df725"
+					(reference "C20")
 					(unit 1)
 				)
@@
 		(dnp no)
 		(fields_autoplaced yes)
-		(property "Reference" "R23"
+		(property "Reference" "R32"
 			(at 199.39 77.4699 0)
 			(effects
@@
 		)
 		(instances
-			(project ""
-				(path "/09377d5d-727f-4ff4-92c8-7a0483d23f1e/b17da045-52ee-4779-bbc6-bef1d0f1615b"
-					(reference "R23")
+			(project "FabOS_MB"
+				(path "/09377d5d-727f-4ff4-92c8-7a0483d23f1e/0151d859-0a6d-4dae-80c2-9bd1219df725"
+					(reference "R32")
 					(unit 1)
 				)
@@
 		(dnp no)
 		(fields_autoplaced yes)
-		(property "Reference" "#PWR021"
+		(property "Reference" "#PWR040"
 			(at 247.65 125.73 0)
 			(effects
@@
 		)
 		(instances
-			(project ""
-				(path "/09377d5d-727f-4ff4-92c8-7a0483d23f1e/b17da045-52ee-4779-bbc6-bef1d0f1615b"
-					(reference "#PWR021")
+			(project "FabOS_MB"
+				(path "/09377d5d-727f-4ff4-92c8-7a0483d23f1e/0151d859-0a6d-4dae-80c2-9bd1219df725"
+					(reference "#PWR040")
 					(unit 1)
 				)
@@
 		(dnp no)
 		(fields_autoplaced yes)
-		(property "Reference" "J1"
+		(property "Reference" "J3"
 			(at 68.58 92.71 0)
 			(effects
@@
 		(instances
 			(project "FabOS_MB"
-				(path "/09377d5d-727f-4ff4-92c8-7a0483d23f1e/b17da045-52ee-4779-bbc6-bef1d0f1615b"
-					(reference "J1")
+				(path "/09377d5d-727f-4ff4-92c8-7a0483d23f1e/0151d859-0a6d-4dae-80c2-9bd1219df725"
+					(reference "J3")
 					(unit 1)
 				)
@@
 		(dnp no)
 		(fields_autoplaced yes)
-		(property "Reference" "C14"
+		(property "Reference" "C21"
 			(at 236.22 104.1462 0)
 			(effects
@@
 		)
 		(instances
-			(project ""
-				(path "/09377d5d-727f-4ff4-92c8-7a0483d23f1e/b17da045-52ee-4779-bbc6-bef1d0f1615b"
-					(reference "C14")
+			(project "FabOS_MB"
+				(path "/09377d5d-727f-4ff4-92c8-7a0483d23f1e/0151d859-0a6d-4dae-80c2-9bd1219df725"
+					(reference "C21")
 					(unit 1)
 				)
@@
 		(dnp no)
 		(fields_autoplaced yes)
-		(property "Reference" "#PWR019"
+		(property "Reference" "#PWR038"
 			(at 68.58 121.92 0)
 			(effects
@@
 		)
 		(instances
-			(project ""
-				(path "/09377d5d-727f-4ff4-92c8-7a0483d23f1e/b17da045-52ee-4779-bbc6-bef1d0f1615b"
-					(reference "#PWR019")
+			(project "FabOS_MB"
+				(path "/09377d5d-727f-4ff4-92c8-7a0483d23f1e/0151d859-0a6d-4dae-80c2-9bd1219df725"
+					(reference "#PWR038")
 					(unit 1)
 				)
@@
 		(dnp no)
 		(fields_autoplaced yes)
-		(property "Reference" "U3"
+		(property "Reference" "U9"
 			(at 213.36 76.2 0)
 			(effects
@@
 		(instances
 			(project "FabOS_MB"
-				(path "/09377d5d-727f-4ff4-92c8-7a0483d23f1e/b17da045-52ee-4779-bbc6-bef1d0f1615b"
-					(reference "U3")
+				(path "/09377d5d-727f-4ff4-92c8-7a0483d23f1e/0151d859-0a6d-4dae-80c2-9bd1219df725"
+					(reference "U9")
 					(unit 1)
 				)
@@
 		(dnp no)
 		(fields_autoplaced yes)
-		(property "Reference" "#PWR020"
+		(property "Reference" "#PWR039"
 			(at 184.15 87.63 0)
 			(effects
@@
 		)
 		(instances
-			(project ""
-				(path "/09377d5d-727f-4ff4-92c8-7a0483d23f1e/b17da045-52ee-4779-bbc6-bef1d0f1615b"
-					(reference "#PWR020")
-					(unit 1)
-				)
+			(project "FabOS_MB"
+				(path "/09377d5d-727f-4ff4-92c8-7a0483d23f1e/0151d859-0a6d-4dae-80c2-9bd1219df725"
+					(reference "#PWR039")
+					(unit 1)
+				)

Commit message: Maj 5V
Parts:
- removed C20: 10µ, symbol Device:C_Small
- added R33: 1k, symbol Device:R
- C21: value 220µ -> 220u
Connections:
- net LIN: now also R33.2
- net TXD: now also U9.4 (TxD)
- net 5V: now reaches U9.7 (VBB)
- net 5V: now also J3.1 (VBUS), R33.1
- net 12V renamed 3.3V
- net 3.3V: no longer J3.1 (VBUS)
Other:
- note removed: "Pour l'alimentation du LIN je n'ai pas compris la doc"
- moved on the sheet: J3

Commit message: Schéma processeur
Parts:
- added R27: 250k, symbol Device:R
- added R28: 125k, symbol Device:R
Connections:
- net EN: now also R27.1
- net GND: now also R27.2, R28.2
- net TXD: now also R28.1

Commit message: Correction de certaines erreurs
Parts:
- renumbered C21 to C20, R27 to R28, R28 to R29, R32 to R30, R33 to R31, U9 to U7
Changed lines of the file:
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@@
 		(dnp no)
 		(fields_autoplaced yes)
-		(property "Reference" "#PWR053"
+		(property "Reference" "#PWR041"
 			(at 182.88 110.49 0)
 			(effects
@@
 			(project ""
 				(path "/09377d5d-727f-4ff4-92c8-7a0483d23f1e/0151d859-0a6d-4dae-80c2-9bd1219df725"
-					(reference "#PWR053")
+					(reference "#PWR041")
 					(unit 1)
 				)
@@
 		(dnp no)
 		(fields_autoplaced yes)
-		(property "Reference" "#PWR054"
+		(property "Reference" "#PWR042"
 			(at 195.58 123.19 0)
 			(effects
@@
 			(project ""
 				(path "/09377d5d-727f-4ff4-92c8-7a0483d23f1e/0151d859-0a6d-4dae-80c2-9bd1219df725"
-					(reference "#PWR054")
+					(reference "#PWR042")
 					(unit 1)
 				)
@@
 		(dnp no)
 		(fields_autoplaced yes)
-		(property "Reference" "R32"
+		(property "Reference" "R30"
 			(at 199.39 77.4699 0)
 			(effects
@@
 			(project "FabOS_MB"
 				(path "/09377d5d-727f-4ff4-92c8-7a0483d23f1e/0151d859-0a6d-4dae-80c2-9bd1219df725"
-					(reference "R32")
+					(reference "R30")
 					(unit 1)
 				)
@@
 		(dnp no)
 		(fields_autoplaced yes)
-		(property "Reference" "R28"
+		(property "Reference" "R29"
 			(at 198.12 111.7599 0)
 			(effects
@@
 			(project ""
 				(path "/09377d5d-727f-4ff4-92c8-7a0483d23f1e/0151d859-0a6d-4dae-80c2-9bd1219df725"
-					(reference "R28")
+					(reference "R29")
 					(unit 1)
 				)
@@
 		(dnp no)
 		(fields_autoplaced yes)
-		(property "Reference" "#PWR040"
+		(property "Reference" "#PWR043"
 			(at 247.65 125.73 0)
 			(effects
@@
 			(project "FabOS_MB"
 				(path "/09377d5d-727f-4ff4-92c8-7a0483d23f1e/0151d859-0a6d-4dae-80c2-9bd1219df725"
-					(reference "#PWR040")
+					(reference "#PWR043")
 					(unit 1)
 				)
@@
 		(dnp no)
 		(fields_autoplaced yes)
-		(property "Reference" "R27"
+		(property "Reference" "R28"
 			(at 185.42 99.0599 0)
 			(effects
@@
 			(project ""
 				(path "/09377d5d-727f-4ff4-92c8-7a0483d23f1e/0151d859-0a6d-4dae-80c2-9bd1219df725"
-					(reference "R27")
+					(reference "R28")
 					(unit 1)
 				)
@@
 		(dnp no)
 		(fields_autoplaced yes)
-		(property "Reference" "C21"
+		(property "Reference" "C20"
 			(at 236.22 104.1462 0)
 			(effects
@@
 			(project "FabOS_MB"
 				(path "/09377d5d-727f-4ff4-92c8-7a0483d23f1e/0151d859-0a6d-4dae-80c2-9bd1219df725"
-					(reference "C21")
+					(reference "C20")
 					(unit 1)
 				)
@@
 		(dnp no)
 		(fields_autoplaced yes)
-		(property "Reference" "#PWR038"
+		(property "Reference" "#PWR040"
 			(at 86.36 123.19 0)
 			(effects
@@
 			(project "FabOS_MB"
 				(path "/09377d5d-727f-4ff4-92c8-7a0483d23f1e/0151d859-0a6d-4dae-80c2-9bd1219df725"
-					(reference "#PWR038")
+					(reference "#PWR040")
 					(unit 1)
 				)
@@
 		(dnp no)
 		(fields_autoplaced yes)
-		(property "Reference" "U9"
+		(property "Reference" "U7"
 			(at 213.36 76.2 0)
 			(effects
@@
 			(project "FabOS_MB"
 				(path "/09377d5d-727f-4ff4-92c8-7a0483d23f1e/0151d859-0a6d-4dae-80c2-9bd1219df725"
-					(reference "U9")
+					(reference "U7")
 					(unit 1)
 				)
@@
 		(dnp no)
 		(fields_autoplaced yes)
-		(property "Reference" "R33"
+		(property "Reference" "R31"
 			(at 236.22 96.5199 0)
 			(effects
@@
 			(project ""
 				(path "/09377d5d-727f-4ff4-92c8-7a0483d23f1e/0151d859-0a6d-4dae-80c2-9bd1219df725"
-					(reference "R33")
-					(unit 1)
-				)
+					(reference "R31")
+					(unit 1)
+				)

Commit message: update pcb
Parts:
- C201: renamed from C20; value 220u -> 1n
- renumbered J3 to J201, R28 to R201, R29 to R202, R30 to R203, R31 to R204, U7 to U201
Connections:
- net 5V: no longer R204.1, U201.7 (VBB)
- net LIN: no longer J201.2 (D-)
- net 3.3V renamed V_MCU
- new net EmergencyStop: J201.2 (D-)
- new net V_LIN: R204.1, U201.7 (VBB)
Other:
- note added: "Pourquoi des résistances de pull-down sur TXD ?"
- moved on the sheet: C201, J201, R201, R202, R203, R204, U201

Commit message: Update pcb
Parts:
- removed R202: 125k, symbol Device:R
Other:
- note removed: "Pourquoi des résistances de pull-down sur TXD ?"
Changed lines of the file:
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@@
-	)
-	(junction
-		(at 104.14 110.49)
-		(diameter 0)
-		(color 0 0 0 0)
 	)
 	(junction
@@
 	(wire
 		(pts
-			(xy 104.14 110.49) (xy 110.49 110.49)
+			(xy 101.6 110.49) (xy 110.49 110.49)
 		)
 		(stroke
@@
 	(wire
 		(pts
-			(xy 101.6 110.49) (xy 104.14 110.49)
-		)
-		(stroke
-			(width 0)
-			(type default)
-		)
-	)
-	(wire
-		(pts
 			(xy 140.97 97.79) (xy 143.51 97.79)
 		)
@@
 			(width 0)
 			(type default)
-		)
-	)
-	(text "Pourquoi des résistances de pull-down sur TXD ?"
-		(exclude_from_sim no)
-		(at 96.52 129.54 0)
-		(effects
-			(font
-				(size 1.27 1.27)
-			)
 		)
 	)
@@
 	)
 	(symbol
-		(lib_id "power:GND")
-		(at 104.14 118.11 0)
-		(unit 1)
-		(exclude_from_sim no)
-		(in_bom yes)
-		(on_board yes)
-		(dnp no)
-		(fields_autoplaced yes)
-		(property "Reference" "#PWR0203"
-			(at 104.14 124.46 0)
-			(effects
-				(font
-					(size 1.27 1.27)
-				)
-				(hide yes)
-			)
-		)
-		(property "Value" "GND"
-			(at 104.14 123.19 0)
-			(effects
-				(font
-					(size 1.27 1.27)
-				)
-			)
-		)
-		(property "Footprint" ""
-			(at 104.14 118.11 0)
-			(effects
-				(font
-					(size 1.27 1.27)
-				)
-				(hide yes)
-			)
-		)
-		(property "Datasheet" ""
-			(at 104.14 118.11 0)
-			(effects
-				(font
-					(size 1.27 1.27)
-				)
-				(hide yes)
-			)
-		)
-		(property "Description" "Power symbol creates a global label with name \"GND\" , ground"
-			(at 104.14 118.11 0)
-			(effects
-				(font
-					(size 1.27 1.27)
-				)
-				(hide yes)
-			)
-		)
-		(pin "1"
-		)
-		(instances
-			(project "FabOS_MB"
-				(path "/09377d5d-727f-4ff4-92c8-7a0483d23f1e/41adeaf0-86bd-4933-9f09-9c5d1e24eb54"
-					(reference "#PWR0203")
-					(unit 1)
-				)
-			)
-		)
-	)
-	(symbol
 		(lib_id "Device:R")
 		(at 104.14 87.63 0)
@@
 					(unit 1)
 				)
-			)
-		)
-	)
-	(symbol
-		(lib_id "Device:R")
-		(at 104.14 114.3 0)
-		(unit 1)
-		(exclude_from_sim no)
-		(in_bom yes)
-		(on_board yes)
-		(dnp no)
-		(fields_autoplaced yes)
-		(property "Reference" "R202"
-			(at 106.68 113.0299 0)
-			(effects
-				(font
-					(size 1.27 1.27)
-				)
-				(justify left)
-			)
-		)
-		(property "Value" "125k"
-			(at 106.68 115.5699 0)
-			(effects
-				(font
-					(size 1.27 1.27)
-				)
-				(justify left)
-			)
-		)
-		(property "Footprint" ""
-			(at 102.362 114.3 90)
-			(effects
-				(font
-					(size 1.27 1.27)
-				)
-				(hide yes)
-			)
-		)
-		(property "Datasheet" "~"
-			(at 104.14 114.3 0)
-			(effects
-				(font
-					(size 1.27 1.27)
-				)
-				(hide yes)
-			)
-		)
-		(property "Description" "Resistor"
-			(at 104.14 114.3 0)
-			(effects
-				(font
-					(size 1.27 1.27)
-				)
-				(hide yes)
-			)
-		)
-		(pin "1"
-		)
-		(pin "2"
-		)
-		(instances
-			(project "FabOS_MB"
-				(path "/09377d5d-727f-4ff4-92c8-7a0483d23f1e/41adeaf0-86bd-4933-9f09-9c5d1e24eb54"
-					(reference "R202")
-					(unit 1)
-				)
