File: FabOS_MB/power.kicad_sch (KiCad schematic)
At the start: 16 parts, among them U1 TPS563201, U2 TDPOWER TAS12-5-W2

Commit message: Update pcb
Parts:
- added D1, D2, D3: LED, symbol Device:LED
- added R28, R29: 5k, symbol Device:R
- added R30: 3k3, symbol Device:R
- D501, D502: value D_Schottky -> BAT60JFILM
Connections:
- net 5V_Flyback: now also D1.2 (A)
- net 5V_USB: now also D2.2 (A)
- net GND: now also R28.2, R29.2, R30.2; no longer U1.1 (GND)
- new net: D3.1 (K), R30.1
- new net: D1.1 (K), R28.1
- new net: D2.1 (K), R29.1
Other:
- note added: "Le faire passer de l'autre côté, ce bn'est qu'attaché à une masse"
- note removed: "EN"
- note removed: "GND"
- note removed: "Refaire le symbole avec les termes utilisés partout dans le monde Phase -> L Neutre -> N Inverser en sortie V+ et V- afin d'avoir le GND en bas"
- note removed: "Refaire le symbole et le schéma du régulateur pour qu'il soit plus lisible Rajouter un commentaire pour le lien entre la tension de sortie et de feedback"
- note removed: "SW"
- note removed: "VBST"
- note removed: "VFB"
- note removed: "VIN"
- moved on the sheet: C1, C2, C3, C4, C5, C6, L1, R1, R2, R3, U1
