File: hardware/FabOS_MB/FabOS_MB.kicad_sch (KiCad schematic)
At the start: 0 parts

Commit message: update pcb
Other:
- sheet LIN ports: added 5V; removed V_LIN
Changed lines of the file:
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@@
+	(wire
+		(pts
+			(xy 203.2 86.36) (xy 215.9 86.36)
+		)
+		(stroke
+			(width 0)
+			(type default)
+		)
+	)
 	(wire
 		(pts
@@
 	(wire
 		(pts
+			(xy 203.2 96.52) (xy 215.9 96.52)
+		)
+		(stroke
+			(width 0)
+			(type default)
+		)
+	)
+	(wire
+		(pts
 			(xy 203.2 91.44) (xy 215.9 91.44)
 		)
@@
 		(pts
 			(xy 203.2 40.64) (xy 215.9 40.64)
-		)
-		(stroke
-			(width 0)
-			(type default)
-		)
-	)
-	(wire
-		(pts
-			(xy 213.36 85.09) (xy 215.9 85.09)
 		)
 		(stroke
@@
 		)
 	)
+	(label "LIN_EN"
+		(at 203.2 86.36 0)
+		(fields_autoplaced yes)
+		(effects
+			(font
+				(size 1.27 1.27)
+			)
+			(justify left bottom)
+		)
+	)
 	(label "ETH_TX_EN"
 		(at 173.99 48.26 180)
@@
 		)
 	)
-	(label "USB_OTG_FS_DP"
-		(at 97.79 48.26 0)
-		(fields_autoplaced yes)
-		(effects
-			(font
-				(size 1.27 1.27)
-			)
-			(justify left bottom)
-		)
-	)
 	(label "ETH_CRS_DV"
 		(at 203.2 55.88 0)
@@
 		)
 	)
-	(label "USB_OTG_DM"
+	(label "USB_DM"
 		(at 173.99 85.09 180)
 		(fields_autoplaced yes)
@@
 		)
 	)
+	(label "ES"
+		(at 203.2 96.52 0)
+		(fields_autoplaced yes)
+		(effects
+			(font
+				(size 1.27 1.27)
+			)
+			(justify left bottom)
+		)
+	)
 	(label "USART1_TX"
 		(at 97.79 36.83 0)
@@
 		)
 	)
-	(label "USB_OTG_DM"
-		(at 97.79 50.8 0)
-		(fields_autoplaced yes)
-		(effects
-			(font
-				(size 1.27 1.27)
-			)
-			(justify left bottom)
-		)
-	)
 	(label "ETH_MDI0"
 		(at 173.99 50.8 180)
@@
 		)
 	)
+	(label "USB_DM"
+		(at 97.79 50.8 0)
+		(fields_autoplaced yes)
+		(effects
+			(font
+				(size 1.27 1.27)
+			)
+			(justify left bottom)
+		)
+	)
 	(label "ETH_TXD0"
 		(at 203.2 40.64 0)
@@
 		)
 	)
-	(label "USB_OTG_FS_DP"
+	(label "USB_DP"
 		(at 173.99 82.55 180)
 		(fields_autoplaced yes)
@@
 	(label "USART1_TX"
 		(at 203.2 93.98 0)
+		(fields_autoplaced yes)
+		(effects
+			(font
+				(size 1.27 1.27)
+			)
+			(justify left bottom)
+		)
+	)
+	(label "USB_DP"
+		(at 97.79 48.26 0)
 		(fields_autoplaced yes)
 		(effects
@@
 	(symbol
 		(lib_id "power:+3.3V")
-		(at 213.36 85.09 90)
-		(unit 1)
-		(exclude_from_sim no)
-		(in_bom yes)
-		(on_board yes)
-		(dnp no)
-		(fields_autoplaced yes)
-		(property "Reference" "#PWR0108"
-			(at 217.17 85.09 0)
-			(effects
-				(font
-					(size 1.27 1.27)
-				)
-				(hide yes)
-			)
-		)
-		(property "Value" "+3.3V"
-			(at 209.55 85.0899 90)
-			(effects
-				(font
-					(size 1.27 1.27)
-				)
-				(justify left)
-			)
-		)
-		(property "Footprint" ""
-			(at 213.36 85.09 0)
-			(effects
-				(font
-					(size 1.27 1.27)
-				)
-				(hide yes)
-			)
-		)
-		(property "Datasheet" ""
-			(at 213.36 85.09 0)
-			(effects
-				(font
-					(size 1.27 1.27)
-				)
-				(hide yes)
-			)
-		)
-		(property "Description" "Power symbol creates a global label with name \"+3.3V\""
-			(at 213.36 85.09 0)
-			(effects
-				(font
-					(size 1.27 1.27)
-				)
-				(hide yes)
-			)
-		)
-		(pin "1"
-		)
-		(instances
-			(project "FabOS_MB"
-				(path "/09377d5d-727f-4ff4-92c8-7a0483d23f1e"
-					(reference "#PWR0108")
-					(unit 1)
-				)
-			)
-		)
-	)
-	(symbol
-		(lib_id "power:+3.3V")
 		(at 213.36 82.55 90)
 		(unit 1)
@@
 		)
 		(pin "EN" input
-			(at 215.9 85.09 180)
+			(at 215.9 86.36 180)
 			(effects
 				(font
@@
 			)
 		)
-		(pin "V_LIN" input
-			(at 215.9 80.01 180)
-			(effects
-				(font
-					(size 1.27 1.27)
-				)
-				(justify left)
-			)
-		)
 		(pin "V_MCU" input
 			(at 215.9 82.55 180)
 			(effects
 				(font
+					(size 1.27 1.27)
+				)
+				(justify left)
+			)
+		)
+		(pin "5V" input
+			(at 215.9 80.01 180)
+			(effects
+				(font

Commit message: PCB_Update
Other:
- sheet STM32 ports: added ES, LIN_EN, NRST_ETH; removed NRST
- sheet ethernet ports: added NRST_LAN8742A; removed NRST
Changed lines of the file:
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@@
+	(wire
+		(pts
+			(xy 97.79 41.91) (xy 114.3 41.91)
+		)
+		(stroke
+			(width 0)
+			(type default)
+		)
+	)
 	(wire
 		(pts
@@
 	(wire
 		(pts
+			(xy 130.81 21.59) (xy 130.81 25.4)
+		)
+		(stroke
+			(width 0)
+			(type default)
+		)
+	)
+	(wire
+		(pts
 			(xy 152.4 40.64) (xy 173.99 40.64)
 		)
@@
 	(wire
 		(pts
-			(xy 97.79 43.18) (xy 114.3 43.18)
-		)
-		(stroke
-			(width 0)
-			(type default)
-		)
-	)
-	(wire
-		(pts
 			(xy 203.2 30.48) (xy 215.9 30.48)
 		)
@@
 		(pts
 			(xy 203.2 93.98) (xy 215.9 93.98)
+		)
+		(stroke
+			(width 0)
+			(type default)
+		)
+	)
+	(wire
+		(pts
+			(xy 133.35 21.59) (xy 133.35 25.4)
 		)
 		(stroke
@@
 		)
 	)
+	(label "ES"
+		(at 130.81 21.59 180)
+		(fields_autoplaced yes)
+		(effects
+			(font
+				(size 1.27 1.27)
+			)
+			(justify right bottom)
+		)
+	)
 	(label "ETH_TXD0"
 		(at 173.99 38.1 180)
@@
 		)
 	)
-	(label "NRST"
-		(at 97.79 43.18 0)
+	(label "NRST_ETH"
+		(at 133.35 21.59 0)
 		(fields_autoplaced yes)
 		(effects
@@
 		)
 	)
-	(label "NRST"
+	(label "NRST_ETH"
 		(at 203.2 59.69 0)
 		(fields_autoplaced yes)
@@
 	(label "ETH_MDC"
 		(at 203.2 45.72 0)
+		(fields_autoplaced yes)
+		(effects
+			(font
+				(size 1.27 1.27)
+			)
+			(justify left bottom)
+		)
+	)
+	(label "LIN_EN"
+		(at 97.79 41.91 0)
 		(fields_autoplaced yes)
 		(effects
@@
 			)
 		)
-		(pin "NRST" bidirectional
-			(at 215.9 59.69 180)
-			(effects
-				(font
-					(size 1.27 1.27)
-				)
-				(justify left)
-			)
-		)
 		(pin "RMII_REF_CLK" output
 			(at 215.9 53.34 180)
@@
 		(pin "RMII_CRS_DV" output
 			(at 215.9 55.88 180)
+			(effects
+				(font
+					(size 1.27 1.27)
+				)
+				(justify left)
+			)
+		)
+		(pin "NRST_LAN8742A" input
+			(at 215.9 59.69 180)
 			(effects
 				(font
@@
 			)
 		)
-		(pin "NRST" input
-			(at 114.3 43.18 180)
-			(effects
-				(font
-					(size 1.27 1.27)
-				)
-				(justify left)
-			)
-		)
+		(pin "LIN_EN" output
+			(at 114.3 41.91 180)
+			(effects
+				(font
+					(size 1.27 1.27)
+				)
+				(justify left)
+			)
+		)
+		(pin "ES" output
+			(at 130.81 25.4 90)
+			(effects
+				(font
+					(size 1.27 1.27)
+				)
+				(justify right)
+			)
+		)
+		(pin "NRST_ETH" output
+			(at 133.35 25.4 90)
+			(effects
+				(font
+					(size 1.27 1.27)
+				)
+				(justify right)
+			)
+		)
