File: hardware/FabOS_MB/STM32.kicad_sch (KiCad schematic)
At the start: 18 parts, among them SW1 boot, SW2 SW_Push, U8 STM32F407VETx

Commit message: update pcb
Parts:
- added C613, C614, C615: 10n, Resistor_SMD:R_0402_1005Metric, symbol Device:C_Small
- added D601, D602, D603: LED, symbol Device:LED
- added R602, R603, R604: R_Small, symbol Device:R_Small
- added R605, R606, R607, R608, R609, R610: 10k, Resistor_SMD:R_0402_1005Metric, symbol Device:R_Small
- added SW603, SW604, SW605: SW_Push, Button_Switch_SMD:SW_Push_1P1T_NO_6x6mm_H9.5mm, symbol Switch:SW_Push
- renumbered C29 to C601, C31 to C602, C33 to C603, C35 to C604, C37 to C605, C39 to C606, C41 to C607, C25 to C608, C26 to C609, C601 to C610, C22 to C611, C27 to C612, C21 to C616, C23 to C617, R32 to R601, SW1 to SW601, SW2 to SW602, U8 to U601
Connections:
- net +3.3V: now also R605.1, R606.1, R607.1
- net GND: now also C613.2, C614.2, C615.2, D601.1 (K), D602.1 (K), D603.1 (K), SW603.1, SW604.1, SW605.1
- new net: R606.2, R609.2, SW604.2
- new net: D601.2 (A), R602.2
- new net: R607.2, R610.2, SW605.2
- new net: D602.2 (A), R603.2
- new net: R605.2, R608.2, SW603.2
- new net: D603.2 (A), R604.2
- new net BTN1: C613.1, R608.1
- new net BTN2: C614.1, R609.1
- new net BTN3: C615.1, R610.1
- new net LED1: R602.1
- new net LED2: R603.1
- new net LED3: R604.1
Other:
- moved on the sheet: C601, C602, C603, C604, C605, C606, C607, C608, C609, C610, C616, C617

Commit message: PCB_Update
Connections:
- net BTN1: now also U601.67 (PA8)
- net BTN2: now also U601.66 (PC9)
- net BTN3: now also U601.65 (PC8)
- net ES: now also U601.60 (PD13)
- net LED1: now also U601.63 (PC6)
- net LED2: now also U601.64 (PC7)
- net LED3: now also U601.62 (PD15)
- net LIN_EN: now also U601.61 (PD14)
- net NRST_ETH: now reaches U601.59 (PD12)
- no-connect marks 69 -> 60
