File: hardware/FabOS_MB/_autosave-FabOS_MB.kicad_sch (KiCad schematic)
At the start: 4 parts

Commit message: update
Other:
- sheet STM32 ports: added USB_OTG_FS_DM; removed USB_OTG_DM
Changed lines of the file:
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@@
-			)
-		)
-		(pin "USB_OTG_DM" bidirectional
-			(at 114.3 45.72 180)
-			(effects
-				(font
-					(size 1.27 1.27)
-				)
-				(justify left)
 			)
 		)
@@
 			(effects
 				(font
+					(size 1.27 1.27)
+				)
+				(justify left)
+			)
+		)
+		(pin "USB_OTG_FS_DM" bidirectional
+			(at 114.3 45.72 180)
+			(effects
+				(font
