File: hardware/FabOS_MB/_autosave-STM32.kicad_sch (KiCad schematic)
At the start: 36 parts, among them SW601 boot, SW602 SW_Push, SW603 SW_Push, SW604 SW_Push, SW605 SW_Push, U601 STM32F407VETx

Commit message: update
Connections:
- net USB_OTG_DM renamed USB_OTG_FS_DM
Changed lines of the file:
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@@
 		)
 	)
-	(hierarchical_label "USB_OTG_DM"
+	(hierarchical_label "USB_OTG_FS_DM"
 		(shape bidirectional)
 		(at 99.06 68.58 0)
