File: hardware/FabOS_MB/power.kicad_sch (KiCad schematic)
At the start: 22 parts, among them U1 TPS563201, U2 TDPOWER TAS12-5-W2

Commit message: update pcb
Parts:
- removed C1, C2: 22u, symbol Device:C_Small
- removed D1, D2, D3: LED, symbol Device:LED
- removed JP501: SolderJumper_2_Bridged, symbol Jumper:SolderJumper_2_Bridged
- removed L1: 2u2, symbol Device:L
- removed R28, R29: 5k, symbol Device:R
- removed R30: 3k3, symbol Device:R
- added C505, C506: 22u, symbol Device:C_Small
- added D503, D504, D505: LED, symbol Device:LED
- added JP501: SolderJumper_2_Open, symbol Jumper:SolderJumper_2_Open
- added L501: 2u2, symbol Device:L
- added R501: 3k3, symbol Device:R
- added R502, R503: 5k, symbol Device:R
- renumbered C5 to C501, C4 to C502, C3 to C503, C6 to C504, R1 to R504, R3 to R505, R2 to R506, U2 to U501, U1 to U502
Connections:
- net 5V_Flyback: now also R503.1
- net 5V_USB: now also R502.1
- net Earth: now also JP501.1 (A)
- net GND: now also U502.1 (GND), C505.2, C506.2, D503.1 (K), D504.1 (K), D505.1 (K), JP501.2 (B)
- net V_out: now also C505.1, C506.1, L501.1
- net at U502.2 (SW): now also C504.2, L501.2; no longer C504.1
- net at U502.6 (VBST): now also C504.1; no longer C504.2
- new net: D505.2 (A), R503.2
- new net: D504.2 (A), R502.2
- new net: D503.2 (A), R501.2
Other:
- note removed: "Le faire passer de l'autre côté, ce bn'est qu'attaché à une masse"
- note removed: "Rajouter des leds sur les alimentations (5V Flyback, 5V USB et 3.3V), Les polariser avec un courant de 1mA max (calculer les résistances de série nécessaire). Trouver une diode schottky qui va bien pour utiliser l'alimentation la plus élevée (pour ne pas voir de problème dans le cas où le cable usb serait branché en même temps que le 230V AC) Sur les nucléos ils utilisent la BAT60JFILM"
- moved on the sheet: C501, C502, C503, C504, D501, D502, R504, R505, R506, U502

Commit message: update
Other:
- moved on the sheet: R501
Changed lines of the file:
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@@
 	(wire
 		(pts
-			(xy 204.47 44.45) (xy 204.47 41.91)
+			(xy 204.47 44.45) (xy 204.47 40.64)
 		)
 		(stroke
@@
 		(pts
 			(xy 120.65 106.68) (xy 120.65 105.41)
-		)
-		(stroke
-			(width 0)
-			(type default)
-		)
-	)
-	(wire
-		(pts
-			(xy 204.47 34.29) (xy 204.47 33.02)
 		)
 		(stroke
@@
 	(symbol
 		(lib_id "Device:R")
-		(at 204.47 38.1 0)
+		(at 204.47 36.83 0)
 		(unit 1)
 		(exclude_from_sim no)
@@
 		(fields_autoplaced yes)
 		(property "Reference" "R501"
-			(at 207.01 36.8299 0)
+			(at 207.01 35.5599 0)
 			(effects
 				(font
@@
 		)
 		(property "Value" "3k3"
-			(at 207.01 39.3699 0)
+			(at 207.01 38.0999 0)
 			(effects
 				(font
@@
 		)
 		(property "Footprint" ""
-			(at 202.692 38.1 90)
+			(at 202.692 36.83 90)
 			(effects
 				(font
@@
 		)
 		(property "Datasheet" "~"
-			(at 204.47 38.1 0)
+			(at 204.47 36.83 0)
 			(effects
 				(font
@@
 		)
 		(property "Description" "Resistor"
-			(at 204.47 38.1 0)
-			(effects
-				(font
+			(at 204.47 36.83 0)
+			(effects
+				(font

Commit message: update
Parts:
- removed R501: 3k3, symbol Device:R
- added R1: 800, symbol Device:R
- R502, R503: value 5k -> 2k3
Connections:
- net at D503.2 (A): now also R1.2
Changed lines of the file:
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@@
-	(wire
-		(pts
-			(xy 204.47 44.45) (xy 204.47 40.64)
-		)
-		(stroke
-			(width 0)
-			(type default)
-		)
-	)
 	(wire
 		(pts
@@
 	(wire
 		(pts
+			(xy 204.47 33.02) (xy 204.47 34.29)
+		)
+		(stroke
+			(width 0)
+			(type default)
+		)
+	)
+	(wire
+		(pts
 			(xy 220.98 120.65) (xy 220.98 119.38)
 		)
@@
 		(pts
 			(xy 210.82 120.65) (xy 210.82 119.38)
+		)
+		(stroke
+			(width 0)
+			(type default)
+		)
+	)
+	(wire
+		(pts
+			(xy 204.47 41.91) (xy 204.47 44.45)
 		)
 		(stroke
@@
 	)
 	(hierarchical_label "5V_USB"
-		(shape output)
+		(shape input)
 		(at 142.24 45.72 180)
 		(fields_autoplaced yes)
@@
 			)
 		)
-		(property "Value" "5k"
+		(property "Value" "2k3"
 			(at 231.14 38.1 90)
 			(effects
@@
 	)
 	(symbol
+		(lib_id "Device:R")
+		(at 204.47 38.1 0)
+		(unit 1)
+		(exclude_from_sim no)
+		(in_bom yes)
+		(on_board yes)
+		(dnp no)
+		(fields_autoplaced yes)
+		(property "Reference" "R1"
+			(at 207.01 36.8299 0)
+			(effects
+				(font
+					(size 1.27 1.27)
+				)
+				(justify left)
+			)
+		)
+		(property "Value" "800"
+			(at 207.01 39.3699 0)
+			(effects
+				(font
+					(size 1.27 1.27)
+				)
+				(justify left)
+			)
+		)
+		(property "Footprint" ""
+			(at 202.692 38.1 90)
+			(effects
+				(font
+					(size 1.27 1.27)
+				)
+				(hide yes)
+			)
+		)
+		(property "Datasheet" "~"
+			(at 204.47 38.1 0)
+			(effects
+				(font
+					(size 1.27 1.27)
+				)
+				(hide yes)
+			)
+		)
+		(property "Description" "Resistor"
+			(at 204.47 38.1 0)
+			(effects
+				(font
+					(size 1.27 1.27)
+				)
+				(hide yes)
+			)
+		)
+		(pin "1"
+		)
+		(pin "2"
+		)
+		(instances
+			(project "FabOS_MB"
+				(path "/09377d5d-727f-4ff4-92c8-7a0483d23f1e/97fc260e-c16c-48c4-b11a-4f8ec3a451f5"
+					(reference "R1")
+					(unit 1)
+				)
+			)
+		)
+	)
+	(symbol
 		(lib_id "power:GND")
 		(at 215.9 54.61 0)
@@
 			)
 		)
-		(property "Value" "5k"
+		(property "Value" "2k3"
 			(at 219.71 38.1 90)
 			(effects
@@
 					(unit 1)
 				)
-			)
-		)
-	)
-	(symbol
-		(lib_id "Device:R")
-		(at 204.47 36.83 0)
-		(unit 1)
-		(exclude_from_sim no)
-		(in_bom yes)
-		(on_board yes)
-		(dnp no)
-		(fields_autoplaced yes)
-		(property "Reference" "R501"
-			(at 207.01 35.5599 0)
-			(effects
-				(font
-					(size 1.27 1.27)
-				)
-				(justify left)
-			)
-		)
-		(property "Value" "3k3"
-			(at 207.01 38.0999 0)
-			(effects
-				(font
-					(size 1.27 1.27)
-				)
-				(justify left)
-			)
-		)
-		(property "Footprint" ""
-			(at 202.692 36.83 90)
-			(effects
-				(font
-					(size 1.27 1.27)
-				)
-				(hide yes)
-			)
-		)
-		(property "Datasheet" "~"
-			(at 204.47 36.83 0)
-			(effects
-				(font
-					(size 1.27 1.27)
-				)
-				(hide yes)
-			)
-		)
-		(property "Description" "Resistor"
-			(at 204.47 36.83 0)
-			(effects
-				(font
-					(size 1.27 1.27)
-				)
-				(hide yes)
-			)
-		)
-		(pin "1"
-		)
-		(pin "2"
-		)
-		(instances
-			(project "FabOS_MB"
-				(path "/09377d5d-727f-4ff4-92c8-7a0483d23f1e/97fc260e-c16c-48c4-b11a-4f8ec3a451f5"
-					(reference "R501")
-					(unit 1)
-				)

Commit message: led
Parts:
- renumbered R504 to R501, R506 to R502, R505 to R503, R1 to R504, R502 to R505, R503 to R506
Changed lines of the file:
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@@
 		(dnp no)
 		(fields_autoplaced yes)
-		(property "Reference" "R503"
+		(property "Reference" "R506"
 			(at 233.68 38.1 90)
 			(effects
@@
 			(project "FabOS_MB"
 				(path "/09377d5d-727f-4ff4-92c8-7a0483d23f1e/97fc260e-c16c-48c4-b11a-4f8ec3a451f5"
-					(reference "R503")
+					(reference "R506")
 					(unit 1)
 				)
@@
 		(on_board yes)
 		(dnp no)
-		(property "Reference" "R504"
+		(property "Reference" "R501"
 			(at 154.94 118.11 90)
 			(effects
@@
 			(project "FabOS_MB"
 				(path "/09377d5d-727f-4ff4-92c8-7a0483d23f1e/97fc260e-c16c-48c4-b11a-4f8ec3a451f5"
-					(reference "R504")
+					(reference "R501")
 					(unit 1)
 				)
@@
 		(dnp no)
 		(fields_autoplaced yes)
-		(property "Reference" "#PWR0507"
+		(property "Reference" "#PWR0513"
 			(at 204.47 60.96 0)
 			(effects
@@
 			(project "FabOS_MB"
 				(path "/09377d5d-727f-4ff4-92c8-7a0483d23f1e/97fc260e-c16c-48c4-b11a-4f8ec3a451f5"
-					(reference "#PWR0507")
+					(reference "#PWR0513")
 					(unit 1)
 				)
@@
 		(dnp no)
 		(fields_autoplaced yes)
-		(property "Reference" "#PWR0504"
+		(property "Reference" "#PWR0506"
 			(at 76.2 45.72 0)
 			(effects
@@
 			(project "FabOS_MB"
 				(path "/09377d5d-727f-4ff4-92c8-7a0483d23f1e/97fc260e-c16c-48c4-b11a-4f8ec3a451f5"
-					(reference "#PWR0504")
+					(reference "#PWR0506")
 					(unit 1)
 				)
@@
 		(dnp no)
 		(fields_autoplaced yes)
-		(property "Reference" "#PWR0516"
+		(property "Reference" "#PWR0511"
 			(at 182.88 135.89 0)
 			(effects
@@
 			(project "FabOS_MB"
 				(path "/09377d5d-727f-4ff4-92c8-7a0483d23f1e/97fc260e-c16c-48c4-b11a-4f8ec3a451f5"
-					(reference "#PWR0516")
+					(reference "#PWR0511")
 					(unit 1)
 				)
@@
 		(dnp no)
 		(fields_autoplaced yes)
-		(property "Reference" "#PWR0513"
+		(property "Reference" "#PWR0509"
 			(at 129.54 120.65 0)
 			(effects
@@
 			(project "FabOS_MB"
 				(path "/09377d5d-727f-4ff4-92c8-7a0483d23f1e/97fc260e-c16c-48c4-b11a-4f8ec3a451f5"
-					(reference "#PWR0513")
+					(reference "#PWR0509")
 					(unit 1)
 				)
@@
 		(on_board yes)
 		(dnp no)
-		(property "Reference" "R505"
+		(property "Reference" "R503"
 			(at 187.706 115.316 90)
 			(effects
@@
 			(project "FabOS_MB"
 				(path "/09377d5d-727f-4ff4-92c8-7a0483d23f1e/97fc260e-c16c-48c4-b11a-4f8ec3a451f5"
-					(reference "R505")
+					(reference "R503")
 					(unit 1)
 				)
@@
 		(dnp no)
 		(fields_autoplaced yes)
-		(property "Reference" "R1"
+		(property "Reference" "R504"
 			(at 207.01 36.8299 0)
 			(effects
@@
 			(project "FabOS_MB"
 				(path "/09377d5d-727f-4ff4-92c8-7a0483d23f1e/97fc260e-c16c-48c4-b11a-4f8ec3a451f5"
-					(reference "R1")
+					(reference "R504")
 					(unit 1)
 				)
@@
 		(dnp no)
 		(fields_autoplaced yes)
-		(property "Reference" "#PWR0508"
+		(property "Reference" "#PWR0514"
 			(at 215.9 60.96 0)
 			(effects
@@
 			(project "FabOS_MB"
 				(path "/09377d5d-727f-4ff4-92c8-7a0483d23f1e/97fc260e-c16c-48c4-b11a-4f8ec3a451f5"
-					(reference "#PWR0508")
+					(reference "#PWR0514")
 					(unit 1)
 				)
@@
 		(dnp no)
 		(fields_autoplaced yes)
-		(property "Reference" "#PWR0514"
+		(property "Reference" "#PWR0515"
 			(at 215.9 128.27 0)
 			(effects
@@
 			(project "FabOS_MB"
 				(path "/09377d5d-727f-4ff4-92c8-7a0483d23f1e/97fc260e-c16c-48c4-b11a-4f8ec3a451f5"
-					(reference "#PWR0514")
+					(reference "#PWR0515")
 					(unit 1)
 				)
@@
 		(dnp no)
 		(fields_autoplaced yes)
-		(property "Reference" "R502"
+		(property "Reference" "R505"
 			(at 222.25 38.1 90)
 			(effects
@@
 			(project "FabOS_MB"
 				(path "/09377d5d-727f-4ff4-92c8-7a0483d23f1e/97fc260e-c16c-48c4-b11a-4f8ec3a451f5"
-					(reference "R502")
+					(reference "R505")
 					(unit 1)
 				)
@@
 		(dnp no)
 		(fields_autoplaced yes)
-		(property "Reference" "#PWR0506"
+		(property "Reference" "#PWR0505"
 			(at 46.99 46.99 0)
 			(effects
@@
 			(project "FabOS_MB"
 				(path "/09377d5d-727f-4ff4-92c8-7a0483d23f1e/97fc260e-c16c-48c4-b11a-4f8ec3a451f5"
-					(reference "#PWR0506")
+					(reference "#PWR0505")
 					(unit 1)
 				)
@@
 		(dnp no)
 		(fields_autoplaced yes)
-		(property "Reference" "#PWR0510"
+		(property "Reference" "#PWR0501"
 			(at 46.99 66.04 0)
 			(effects
@@
 			(project "FabOS_MB"
 				(path "/09377d5d-727f-4ff4-92c8-7a0483d23f1e/97fc260e-c16c-48c4-b11a-4f8ec3a451f5"
-					(reference "#PWR0510")
+					(reference "#PWR0501")
 					(unit 1)
 				)
@@
 		(dnp no)
 		(fields_autoplaced yes)
-		(property "Reference" "#PWR0515"
+		(property "Reference" "#PWR0510"
 			(at 170.18 135.89 0)
 			(effects
@@
 			(project "FabOS_MB"
 				(path "/09377d5d-727f-4ff4-92c8-7a0483d23f1e/97fc260e-c16c-48c4-b11a-4f8ec3a451f5"
-					(reference "#PWR0515")
+					(reference "#PWR0510")
 					(unit 1)
 				)
@@
 		(on_board yes)
 		(dnp no)
-		(property "Reference" "R506"
+		(property "Reference" "R502"
 			(at 184.404 124.46 0)
 			(effects
@@
 			(project "FabOS_MB"
 				(path "/09377d5d-727f-4ff4-92c8-7a0483d23f1e/97fc260e-c16c-48c4-b11a-4f8ec3a451f5"
-					(reference "R506")
+					(reference "R502")
 					(unit 1)
 				)
@@
 		(dnp no)
 		(fields_autoplaced yes)
-		(property "Reference" "#PWR0505"
+		(property "Reference" "#PWR0507"
 			(at 88.9 45.72 0)
 			(effects
@@
 			(project "FabOS_MB"
 				(path "/09377d5d-727f-4ff4-92c8-7a0483d23f1e/97fc260e-c16c-48c4-b11a-4f8ec3a451f5"
-					(reference "#PWR0505")
+					(reference "#PWR0507")
 					(unit 1)
 				)
@@
 		(dnp no)
 		(fields_autoplaced yes)
-		(property "Reference" "#PWR0509"
+		(property "Reference" "#PWR0516"
 			(at 227.33 60.96 0)
 			(effects
@@
 			(project "FabOS_MB"
 				(path "/09377d5d-727f-4ff4-92c8-7a0483d23f1e/97fc260e-c16c-48c4-b11a-4f8ec3a451f5"
-					(reference "#PWR0509")
+					(reference "#PWR0516")
 					(unit 1)
 				)
@@
 		(dnp no)
 		(fields_autoplaced yes)
-		(property "Reference" "#PWR0511"
+		(property "Reference" "#PWR0502"
 			(at 46.99 76.2 0)
 			(effects
@@
 			(project "FabOS_MB"
 				(path "/09377d5d-727f-4ff4-92c8-7a0483d23f1e/97fc260e-c16c-48c4-b11a-4f8ec3a451f5"
-					(reference "#PWR0511")
+					(reference "#PWR0502")
 					(unit 1)
 				)
@@
 		(dnp no)
 		(fields_autoplaced yes)
-		(property "Reference" "#PWR0501"
+		(property "Reference" "#PWR0512"
 			(at 204.47 36.83 0)
 			(effects
@@
 			(project ""
 				(path "/09377d5d-727f-4ff4-92c8-7a0483d23f1e/97fc260e-c16c-48c4-b11a-4f8ec3a451f5"
-					(reference "#PWR0501")
+					(reference "#PWR0512")
 					(unit 1)
 				)
@@
 		(dnp no)
 		(fields_autoplaced yes)
-		(property "Reference" "#PWR0503"
+		(property "Reference" "#PWR0504"
 			(at 43.18 38.1 0)
 			(effects
@@
 			(project "FabOS_MB"
 				(path "/09377d5d-727f-4ff4-92c8-7a0483d23f1e/97fc260e-c16c-48c4-b11a-4f8ec3a451f5"
-					(reference "#PWR0503")
+					(reference "#PWR0504")
 					(unit 1)
 				)
@@
 		(dnp no)
 		(fields_autoplaced yes)
-		(property "Reference" "#PWR0512"
+		(property "Reference" "#PWR0508"
 			(at 90.17 82.55 0)
 			(effects
@@
 			(project "FabOS_MB"
 				(path "/09377d5d-727f-4ff4-92c8-7a0483d23f1e/97fc260e-c16c-48c4-b11a-4f8ec3a451f5"
-					(reference "#PWR0512")
+					(reference "#PWR0508")
 					(unit 1)
 				)
@@
 		(dnp no)
 		(fields_autoplaced yes)
-		(property "Reference" "#PWR0502"
+		(property "Reference" "#PWR0503"
 			(at 43.18 35.56 0)
 			(effects
@@
 			(project "FabOS_MB"
 				(path "/09377d5d-727f-4ff4-92c8-7a0483d23f1e/97fc260e-c16c-48c4-b11a-4f8ec3a451f5"
-					(reference "#PWR0502")
-					(unit 1)
-				)
+					(reference "#PWR0503")
+					(unit 1)
+				)

Commit message: Correction des dernières erreurs
Parts:
- R504: value 800 -> 2k3
Changed lines of the file:
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@@
+	)
+	(symbol
+		(lib_id "Device:R")
+		(at 215.9 38.1 0)
+		(unit 1)
+		(exclude_from_sim no)
+		(in_bom yes)
+		(on_board yes)
+		(dnp no)
+		(fields_autoplaced yes)
+		(property "Reference" "R505"
+			(at 222.25 38.1 90)
+			(effects
+				(font
+					(size 1.27 1.27)
+				)
+			)
+		)
+		(property "Value" "2k3"
+			(at 219.71 38.1 90)
+			(effects
+				(font
+					(size 1.27 1.27)
+				)
+			)
+		)
+		(property "Footprint" ""
+			(at 214.122 38.1 90)
+			(effects
+				(font
+					(size 1.27 1.27)
+				)
+				(hide yes)
+			)
+		)
+		(property "Datasheet" "~"
+			(at 215.9 38.1 0)
+			(effects
+				(font
+					(size 1.27 1.27)
+				)
+				(hide yes)
+			)
+		)
+		(property "Description" "Resistor"
+			(at 215.9 38.1 0)
+			(effects
+				(font
+					(size 1.27 1.27)
+				)
+				(hide yes)
+			)
+		)
+		(pin "1"
+		)
+		(pin "2"
+		)
+		(instances
+			(project "FabOS_MB"
+				(path "/09377d5d-727f-4ff4-92c8-7a0483d23f1e/97fc260e-c16c-48c4-b11a-4f8ec3a451f5"
+					(reference "R505")
+					(unit 1)
+				)
+			)
+		)
 	)
 	(symbol
@@
 	)
 	(symbol
+		(lib_id "Device:R")
+		(at 204.47 38.1 0)
+		(unit 1)
+		(exclude_from_sim no)
+		(in_bom yes)
+		(on_board yes)
+		(dnp no)
+		(fields_autoplaced yes)
+		(property "Reference" "R504"
+			(at 210.82 38.1 90)
+			(effects
+				(font
+					(size 1.27 1.27)
+				)
+			)
+		)
+		(property "Value" "2k3"
+			(at 208.28 38.1 90)
+			(effects
+				(font
+					(size 1.27 1.27)
+				)
+			)
+		)
+		(property "Footprint" ""
+			(at 202.692 38.1 90)
+			(effects
+				(font
+					(size 1.27 1.27)
+				)
+				(hide yes)
+			)
+		)
+		(property "Datasheet" "~"
+			(at 204.47 38.1 0)
+			(effects
+				(font
+					(size 1.27 1.27)
+				)
+				(hide yes)
+			)
+		)
+		(property "Description" "Resistor"
+			(at 204.47 38.1 0)
+			(effects
+				(font
+					(size 1.27 1.27)
+				)
+				(hide yes)
+			)
+		)
+		(pin "1"
+		)
+		(pin "2"
+		)
+		(instances
+			(project "FabOS_MB"
+				(path "/09377d5d-727f-4ff4-92c8-7a0483d23f1e/97fc260e-c16c-48c4-b11a-4f8ec3a451f5"
+					(reference "R504")
+					(unit 1)
+				)
+			)
+		)
+	)
+	(symbol
 		(lib_id "Jumper:SolderJumper_2_Open")
 		(at 82.55 36.83 0)
@@
 	)
 	(symbol
-		(lib_id "Device:R")
-		(at 204.47 38.1 0)
-		(unit 1)
-		(exclude_from_sim no)
-		(in_bom yes)
-		(on_board yes)
-		(dnp no)
-		(fields_autoplaced yes)
-		(property "Reference" "R504"
-			(at 207.01 36.8299 0)
-			(effects
-				(font
-					(size 1.27 1.27)
-				)
-				(justify left)
-			)
-		)
-		(property "Value" "800"
-			(at 207.01 39.3699 0)
-			(effects
-				(font
-					(size 1.27 1.27)
-				)
-				(justify left)
-			)
-		)
-		(property "Footprint" ""
-			(at 202.692 38.1 90)
-			(effects
-				(font
-					(size 1.27 1.27)
-				)
-				(hide yes)
-			)
-		)
-		(property "Datasheet" "~"
-			(at 204.47 38.1 0)
-			(effects
-				(font
-					(size 1.27 1.27)
-				)
-				(hide yes)
-			)
-		)
-		(property "Description" "Resistor"
-			(at 204.47 38.1 0)
-			(effects
-				(font
-					(size 1.27 1.27)
-				)
-				(hide yes)
-			)
-		)
-		(pin "1"
-		)
-		(pin "2"
-		)
-		(instances
-			(project "FabOS_MB"
-				(path "/09377d5d-727f-4ff4-92c8-7a0483d23f1e/97fc260e-c16c-48c4-b11a-4f8ec3a451f5"
-					(reference "R504")
-					(unit 1)
-				)
-			)
-		)
-	)
-	(symbol
 		(lib_id "power:GND")
 		(at 215.9 54.61 0)
@@
 					(unit 1)
 				)
-			)
-		)
-	)
-	(symbol
-		(lib_id "Device:R")
-		(at 215.9 38.1 0)
-		(unit 1)
-		(exclude_from_sim no)
-		(in_bom yes)
-		(on_board yes)
-		(dnp no)
-		(fields_autoplaced yes)
-		(property "Reference" "R505"
-			(at 222.25 38.1 90)
-			(effects
-				(font
-					(size 1.27 1.27)
-				)
-			)
-		)
-		(property "Value" "2k3"
-			(at 219.71 38.1 90)
-			(effects
-				(font
-					(size 1.27 1.27)
-				)
-			)
-		)
-		(property "Footprint" ""
-			(at 214.122 38.1 90)
-			(effects
-				(font
-					(size 1.27 1.27)
-				)
-				(hide yes)
-			)
-		)
-		(property "Datasheet" "~"
-			(at 215.9 38.1 0)
-			(effects
-				(font
-					(size 1.27 1.27)
-				)
-				(hide yes)
-			)
-		)
-		(property "Description" "Resistor"
-			(at 215.9 38.1 0)
-			(effects
-				(font
-					(size 1.27 1.27)
-				)
-				(hide yes)
-			)
-		)
-		(pin "1"
-		)
-		(pin "2"
-		)
-		(instances
-			(project "FabOS_MB"
-				(path "/09377d5d-727f-4ff4-92c8-7a0483d23f1e/97fc260e-c16c-48c4-b11a-4f8ec3a451f5"
-					(reference "R505")
-					(unit 1)
-				)

Commit message: 800 ohms
Parts:
- R504: value 2k3 -> 800
Changed lines of the file:
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@@
 		(fields_autoplaced yes)
 		(property "Reference" "R504"
-			(at 210.82 38.1 90)
+			(at 207.01 36.8299 0)
 			(effects
 				(font
 					(size 1.27 1.27)
 				)
+				(justify left)
 			)
 		)
-		(property "Value" "2k3"
-			(at 208.28 38.1 90)
+		(property "Value" "800"
+			(at 207.01 39.3699 0)
 			(effects
 				(font
 					(size 1.27 1.27)
 				)
+				(justify left)
 			)
 		)

Commit message: connecteur programmation
Changed lines of the file:
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@@
+	(wire
+		(pts
+			(xy 204.47 41.91) (xy 204.47 44.45)
+		)
+		(stroke
+			(width 0)
+			(type default)
+		)
+	)
 	(wire
 		(pts
@@
 	(wire
 		(pts
-			(xy 204.47 33.02) (xy 204.47 34.29)
-		)
-		(stroke
-			(width 0)
-			(type default)
-		)
-	)
-	(wire
-		(pts
 			(xy 220.98 120.65) (xy 220.98 119.38)
 		)
@@
 	(wire
 		(pts
-			(xy 204.47 41.91) (xy 204.47 44.45)
-		)
-		(stroke
-			(width 0)
-			(type default)
-		)
-	)
-	(wire
-		(pts
 			(xy 120.65 105.41) (xy 129.54 105.41)
 		)
@@
 		(pts
 			(xy 120.65 106.68) (xy 120.65 105.41)
+		)
+		(stroke
+			(width 0)
+			(type default)
+		)
+	)
+	(wire
+		(pts
+			(xy 204.47 29.21) (xy 204.47 34.29)
 		)
 		(stroke
@@
 	)
 	(symbol
-		(lib_id "Device:R")
-		(at 204.47 38.1 0)
-		(unit 1)
-		(exclude_from_sim no)
-		(in_bom yes)
-		(on_board yes)
-		(dnp no)
-		(fields_autoplaced yes)
-		(property "Reference" "R504"
-			(at 207.01 36.8299 0)
-			(effects
-				(font
-					(size 1.27 1.27)
-				)
-				(justify left)
-			)
-		)
-		(property "Value" "800"
-			(at 207.01 39.3699 0)
-			(effects
-				(font
-					(size 1.27 1.27)
-				)
-				(justify left)
-			)
-		)
-		(property "Footprint" ""
-			(at 202.692 38.1 90)
-			(effects
-				(font
-					(size 1.27 1.27)
-				)
-				(hide yes)
-			)
-		)
-		(property "Datasheet" "~"
-			(at 204.47 38.1 0)
-			(effects
-				(font
-					(size 1.27 1.27)
-				)
-				(hide yes)
-			)
-		)
-		(property "Description" "Resistor"
-			(at 204.47 38.1 0)
-			(effects
-				(font
-					(size 1.27 1.27)
-				)
-				(hide yes)
-			)
-		)
-		(pin "1"
-		)
-		(pin "2"
-		)
-		(instances
-			(project "FabOS_MB"
-				(path "/09377d5d-727f-4ff4-92c8-7a0483d23f1e/97fc260e-c16c-48c4-b11a-4f8ec3a451f5"
-					(reference "R504")
-					(unit 1)
-				)
-			)
-		)
-	)
-	(symbol
 		(lib_id "Jumper:SolderJumper_2_Open")
 		(at 82.55 36.83 0)
@@
 	)
 	(symbol
+		(lib_id "Device:R")
+		(at 204.47 38.1 0)
+		(unit 1)
+		(exclude_from_sim no)
+		(in_bom yes)
+		(on_board yes)
+		(dnp no)
+		(fields_autoplaced yes)
+		(property "Reference" "R504"
+			(at 207.01 36.8299 0)
+			(effects
+				(font
+					(size 1.27 1.27)
+				)
+				(justify left)
+			)
+		)
+		(property "Value" "800"
+			(at 207.01 39.3699 0)
+			(effects
+				(font
+					(size 1.27 1.27)
+				)
+				(justify left)
+			)
+		)
+		(property "Footprint" ""
+			(at 202.692 38.1 90)
+			(effects
+				(font
+					(size 1.27 1.27)
+				)
+				(hide yes)
+			)
+		)
+		(property "Datasheet" "~"
+			(at 204.47 38.1 0)
+			(effects
+				(font
+					(size 1.27 1.27)
+				)
+				(hide yes)
+			)
+		)
+		(property "Description" "Resistor"
+			(at 204.47 38.1 0)
+			(effects
+				(font
+					(size 1.27 1.27)
+				)
+				(hide yes)
+			)
+		)
+		(pin "1"
+		)
+		(pin "2"
+		)
+		(instances
+			(project "FabOS_MB"
+				(path "/09377d5d-727f-4ff4-92c8-7a0483d23f1e/97fc260e-c16c-48c4-b11a-4f8ec3a451f5"
+					(reference "R504")
+					(unit 1)
+				)
+			)
+		)
+	)
+	(symbol
 		(lib_id "Device:C_Small")
 		(at 120.65 109.22 180)
@@
 	(symbol
 		(lib_id "power:+3.3V")
-		(at 204.47 33.02 0)
+		(at 204.47 29.21 0)
 		(unit 1)
 		(exclude_from_sim no)
@@
 		(fields_autoplaced yes)
 		(property "Reference" "#PWR0512"
-			(at 204.47 36.83 0)
+			(at 204.47 33.02 0)
 			(effects
 				(font
@@
 		)
 		(property "Value" "+3.3V"
-			(at 204.47 27.94 0)
-			(effects
-				(font
-					(size 1.27 1.27)
-				)
-			)
-		)
-		(property "Footprint" ""
-			(at 204.47 33.02 0)
+			(at 204.47 24.13 0)
+			(effects
+				(font
+					(size 1.27 1.27)
+				)
+			)
+		)
+		(property "Footprint" ""
+			(at 204.47 29.21 0)
 			(effects
 				(font
@@
 		)
 		(property "Datasheet" ""
-			(at 204.47 33.02 0)
+			(at 204.47 29.21 0)
 			(effects
 				(font
@@
 		)
 		(property "Description" "Power symbol creates a global label with name \"+3.3V\""
-			(at 204.47 33.02 0)
-			(effects
-				(font
+			(at 204.47 29.21 0)
+			(effects
+				(font
