File: hardware/FabOS_MB/power.kicad_sch (KiCad schematic)
At the start: 22 parts, among them U501 TDPOWER TAS12-5-W2, U502 TPS563201

Commit message: Updare pcb
Parts:
- C501, C504: footprint (none) -> Capacitor_SMD:C_0402_1005Metric
- C502, C503: footprint (none) -> Capacitor_SMD:C_Elec_4x5.4; LCSC (none) -> C213487; MPN (none) -> VT1C100M0405; Matériau Céramique -> (none)
- C505: footprint (none) -> Capacitor_SMD:C_Elec_6.3x5.4; LCSC (none) -> C72505; MPN (none) -> RVT1H220M0605
- C506: footprint (none) -> Capacitor_SMD:C_Elec_6.3x5.4
- D501, D502: footprint (none) -> Diode_SMD:D_SOD-323
- D503, D504, D505: footprint (none) -> Diode_SMD:D_0402_1005Metric
- JP501: footprint (none) -> Jumper:SolderJumper-2_P1.3mm_Open_Pad1.0x1.5mm
- L501: footprint (none) -> Inductor_SMD:L_0402_1005Metric
- R501, R502, R503, R504, R505, R506: footprint (none) -> Resistor_SMD:R_0402_1005Metric
Connections:
- net 5V_max: now also C502.1, C503.1; no longer C502.2, C503.2
- net GND: now also C502.2, C503.2; no longer C502.1, C503.1
