File: hardware/FabOS_MB/ethernet.kicad_sch (KiCad schematic)
At the start: 43 parts, among them J1 RJ45, U3 LAN8742A, U4 USBLC6-4SC6, U5 CND-tek B1601S, Y1 Crystal_GND24

Commit message: update pcb
Parts:
- removed C13: 1uF_X5R_0603, symbol Device:C_Small
- removed C14: 470p, symbol Device:C_Small
- removed C15, C16, C17, C18: 100n, symbol Device:C_Small
- removed FB1: FerriteBead_Small, symbol Device:FerriteBead_Small
- removed JP1: Jumper_2_Small_Bridged, symbol Jumper:Jumper_2_Small_Bridged
- removed JP2, JP3: Jumper_2_Small_Open, symbol Jumper:Jumper_2_Small_Open
- removed R23: 270, symbol Device:R_Small
- removed U4: USBLC6-4SC6, Package_TO_SOT_SMD:SOT-23-6, symbol Power_Protection:USBLC6-4SC6
- added C301: 470p, symbol Device:C_Small
- added C302: 1u, symbol Device:C_Small
- added C303, C304, C305, C309: 100n, symbol Device:C_Small
- added FB301: FerriteBead_Small, symbol Device:FerriteBead_Small
- added R314: 270, symbol Device:R_Small
- added U301: USBLC6-4SC6, Package_TO_SOT_SMD:SOT-23-6, symbol Power_Protection:USBLC6-4SC6
- C310: renamed from C19; value TC1206KKX7RDBB102 -> 1n; Ref ST (none) -> TC1206KKX7RDBB102
- renumbered C10 to C306, C11 to C307, C12 to C308, C8 to C311, C9 to C312, J1 to J301, R14 to R301, R15 to R302, R16 to R303, R17 to R304, R9 to R305, R11 to R306, R12 to R307, R24 to R308, R25 to R309, R5 to R310, R7 to R311, R13 to R312, R4 to R313, R18 to R315, R8 to R316, R19 to R317, R20 to R318, R21 to R319, R22 to R320, R6 to R321, R10 to R322, U3 to U302, U5 to U303, Y1 to Y301
Connections:
- net +3.3V: now also C303.2, FB301.1
- net CT: now also C304.1, C305.1, C309.1, FB301.2, U301.5 (VBUS)
- net Earth: now also C310.2, C309.2, U301.2 (GND)
- net GND: now also C301.1, C302.2, C303.1, C304.2, C305.2, R314.2; no longer C310.2
- net TD+: now reaches R301.2, U302.21 (TXP), U303.1 (TD+)
- net TD+: now also U301.1 (I/O1); no longer R302.1, R303.1, R304.1
- net at J301.9 (LED1-): now also R314.1
- net at C312.2, U302.4 (XTAL2): now also Y301.3; no longer Y301.1
- net RD+: now reaches U302.23 (RXP), U303.6 (RD+)
- net RD+: now also R303.1, U301.4 (I/O3)
- net TD-: now reaches U302.20 (TXN), U303.3 (TD-)
- net TD-: now also R302.1, U301.3 (I/O2)
- net RD-: now reaches U302.22 (RXN), U303.8 (RD-)
- net RD-: now also R304.1, U301.6 (I/O4)
- net NRST_LAN8742A: now reaches U302.15 (~{RST})
- net at C311.2, U302.5 (XTAL1/CLKIN): now also Y301.1; no longer Y301.3
- net VCCR renamed VDDCR
- net VDDCR: now also C301.2, C302.1
Other:
- note added: "Crystals are not polarized"
- note added: "Decoupling capacitor CT"
- note added: "Decoupling capacitor VDDA 1x 100nF per VDDA input"
- note added: "Diff Pair 100 ohm"
- note added: "EFI Capacitor, 2kV"
- note added: "ESD pin can be swaped for easier routing"
- note added: "For internal LDO regulator +1.2V"
- note removed: "!!! certains condos ont des noms particuliers"
- note removed: "2 Label pour le meme net, il faut faire un choix"
- note removed: "C'est un quartz ou un oscillateur ?"
- note removed: "ERREUR ?"
- note removed: "Le NRST ne doit pas être le même que celui du processeur, renommer le NRST du PHY en NRST_LAN8742A et le relier à un GPIO du stm32"
- note removed: "TX P N en paire différentielle 100ohm RX P N en paire différentielle 100ohm"
- note removed: "besoin oscillateur crystal X53T-C20SSA-25.000MHz"
- moved on the sheet: C306, C307, C308, C310, C311, C312, J301, R301, R302, R303, R304, R305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

Commit message: update
Changed lines of the file:
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@@
 	)
 	(junction
+		(at 88.9 33.02)
+		(diameter 0)
+		(color 0 0 0 0)
+	)
+	(junction
 		(at 107.95 64.77)
 		(diameter 0)
@@
 	)
 	(junction
+		(at 57.15 27.94)
+		(diameter 0)
+		(color 0 0 0 0)
+	)
+	(junction
 		(at 74.93 140.97)
 		(diameter 0)
@@
 	(wire
 		(pts
+			(xy 204.47 87.63) (xy 199.39 87.63)
+		)
+		(stroke
+			(width 0)
+			(type default)
+		)
+	)
+	(wire
+		(pts
 			(xy 135.89 33.02) (xy 125.73 33.02)
 		)
@@
 	(wire
 		(pts
+			(xy 199.39 91.44) (xy 204.47 91.44)
+		)
+		(stroke
+			(width 0)
+			(type default)
+		)
+	)
+	(wire
+		(pts
 			(xy 278.13 91.44) (xy 275.59 91.44)
 		)
@@
 	(wire
 		(pts
+			(xy 57.15 27.94) (xy 57.15 31.75)
+		)
+		(stroke
+			(width 0)
+			(type default)
+		)
+	)
+	(wire
+		(pts
 			(xy 66.04 138.43) (xy 66.04 140.97)
 		)
@@
 	(wire
 		(pts
-			(xy 204.47 90.17) (xy 199.39 90.17)
-		)
-		(stroke
-			(width 0)
-			(type default)
-		)
-	)
-	(wire
-		(pts
 			(xy 234.95 107.95) (xy 234.95 105.41)
 		)
@@
 	(wire
 		(pts
-			(xy 199.39 107.95) (xy 204.47 107.95)
+			(xy 199.39 110.49) (xy 204.47 110.49)
 		)
 		(stroke
@@
 	(wire
 		(pts
+			(xy 88.9 33.02) (xy 97.79 33.02)
+		)
+		(stroke
+			(width 0)
+			(type default)
+		)
+	)
+	(wire
+		(pts
 			(xy 215.9 107.95) (xy 215.9 105.41)
 		)
@@
 	(wire
 		(pts
-			(xy 57.15 26.67) (xy 57.15 31.75)
+			(xy 57.15 26.67) (xy 57.15 27.94)
 		)
 		(stroke
@@
 	(wire
 		(pts
-			(xy 86.36 33.02) (xy 97.79 33.02)
+			(xy 86.36 33.02) (xy 88.9 33.02)
 		)
 		(stroke
@@
 	(wire
 		(pts
+			(xy 204.47 106.68) (xy 204.47 105.41)
+		)
+		(stroke
+			(width 0)
+			(type default)
+		)
+	)
+	(wire
+		(pts
 			(xy 146.05 81.28) (xy 146.05 91.44)
 		)
@@
 	(wire
 		(pts
-			(xy 199.39 105.41) (xy 204.47 105.41)
+			(xy 199.39 106.68) (xy 204.47 106.68)
 		)
 		(stroke
@@
 	(wire
 		(pts
-			(xy 199.39 82.55) (xy 204.47 82.55)
+			(xy 199.39 83.82) (xy 204.47 83.82)
 		)
 		(stroke
@@
 	(wire
 		(pts
-			(xy 199.39 86.36) (xy 204.47 86.36)
-		)
-		(stroke
-			(width 0)
-			(type default)
-		)
-	)
-	(wire
-		(pts
 			(xy 236.22 83.82) (xy 240.03 83.82)
 		)
@@
 	)
 	(rectangle
-		(start 199.39 86.995)
-		(end 205.105 91.44)
+		(start 199.39 88.265)
+		(end 205.105 92.71)
 		(stroke
 			(width 0)
@@
 	)
 	(rectangle
-		(start 199.39 79.375)
-		(end 205.105 83.82)
+		(start 199.39 80.645)
+		(end 205.105 85.09)
 		(stroke
 			(width 0)
@@
 	)
 	(rectangle
-		(start 199.39 104.775)
-		(end 205.105 109.22)
+		(start 199.39 107.315)
+		(end 205.105 111.76)
 		(stroke
 			(width 0)
@@
 	)
 	(rectangle
-		(start 46.99 17.78)
-		(end 66.675 42.545)
+		(start 43.18 17.78)
+		(end 65.405 42.545)
 		(stroke
 			(width 0)
@@
 	(text "For internal LDO \nregulator +1.2V"
 		(exclude_from_sim no)
-		(at 57.15 21.59 0)
+		(at 54.864 21.59 0)
 		(effects
 			(font
@@
 	)
 	(label "TX+"
-		(at 204.47 82.55 180)
-		(fields_autoplaced yes)
-		(effects
-			(font
-				(size 1.27 1.27)
-			)
-			(justify right bottom)
-		)
-	)
-	(label "TX-"
-		(at 204.47 90.17 180)
+		(at 204.47 83.82 180)
 		(fields_autoplaced yes)
 		(effects
@@
 	)
 	(label "TXCT"
-		(at 204.47 86.36 180)
+		(at 204.47 87.63 180)
 		(fields_autoplaced yes)
 		(effects
@@
 	)
 	(label "RXCT"
-		(at 204.47 105.41 180)
+		(at 204.47 106.68 180)
 		(fields_autoplaced yes)
 		(effects
@@
 		)
 	)
+	(label "TX-"
+		(at 204.47 91.44 180)
+		(fields_autoplaced yes)
+		(effects
+			(font
+				(size 1.27 1.27)
+			)
+			(justify right bottom)
+		)
+	)
 	(label "RXCT"
 		(at 215.9 93.98 270)
@@
 	)
 	(label "RX-"
-		(at 204.47 107.95 180)
+		(at 204.47 110.49 180)
 		(fields_autoplaced yes)
 		(effects
@@
 	)
 	(symbol
+		(lib_id "power:PWR_FLAG")
+		(at 88.9 33.02 180)
+		(unit 1)
+		(exclude_from_sim no)
+		(in_bom yes)
+		(on_board yes)
+		(dnp no)
+		(fields_autoplaced yes)
+		(property "Reference" "#FLG03"
+			(at 88.9 34.925 0)
+			(effects
+				(font
+					(size 1.27 1.27)
+				)
+				(hide yes)
+			)
+		)
+		(property "Value" "PWR_FLAG"
+			(at 88.9 38.1 0)
+			(effects
+				(font
+					(size 1.27 1.27)
+				)
+			)
+		)
+		(property "Footprint" ""
+			(at 88.9 33.02 0)
+			(effects
+				(font
+					(size 1.27 1.27)
+				)
+				(hide yes)
+			)
+		)
+		(property "Datasheet" "~"
+			(at 88.9 33.02 0)
+			(effects
+				(font
+					(size 1.27 1.27)
+				)
+				(hide yes)
+			)
+		)
+		(property "Description" "Special symbol for telling ERC where power comes from"
+			(at 88.9 33.02 0)
+			(effects
+				(font
+					(size 1.27 1.27)
+				)
+				(hide yes)
+			)
+		)
+		(pin "1"
+		)
+		(instances
+			(project ""
+				(path "/09377d5d-727f-4ff4-92c8-7a0483d23f1e/97c1e665-4fec-464e-b9f4-4fa619e0ae43"
+					(reference "#FLG03")
+					(unit 1)
+				)
+			)
+		)
+	)
+	(symbol
 		(lib_id "Device:R_Small")
 		(at 271.78 96.52 90)
@@
 					(unit 1)
 				)
+			)
+		)
+	)
+	(symbol
+		(lib_id "power:PWR_FLAG")
+		(at 57.15 27.94 90)
+		(unit 1)
+		(exclude_from_sim no)
+		(in_bom yes)
+		(on_board yes)
+		(dnp no)
+		(fields_autoplaced yes)
+		(property "Reference" "#FLG04"
+			(at 55.245 27.94 0)
+			(effects
+				(font
+					(size 1.27 1.27)
+				)
+				(hide yes)
+			)
+		)
+		(property "Value" "PWR_FLAG"
+			(at 53.34 27.9399 90)
+			(effects
+				(font
+					(size 1.27 1.27)
+				)
+				(justify left)
+			)
+		)
+		(property "Footprint" ""
+			(at 57.15 27.94 0)
+			(effects
+				(font
+					(size 1.27 1.27)
+				)
+				(hide yes)
+			)
+		)
+		(property "Datasheet" "~"
+			(at 57.15 27.94 0)
+			(effects
+				(font
+					(size 1.27 1.27)
+				)
+				(hide yes)
+			)
+		)
+		(property "Description" "Special symbol for telling ERC where power comes from"
+			(at 57.15 27.94 0)
+			(effects
+				(font
+					(size 1.27 1.27)
+				)
+				(hide yes)
+			)
+		)
+		(pin "1"
+		)
+		(instances
+			(project ""
+				(path "/09377d5d-727f-4ff4-92c8-7a0483d23f1e/97c1e665-4fec-464e-b9f4-4fa619e0ae43"
+					(reference "#FLG04")
+					(unit 1)
+				)

Commit message: led
Parts:
- renumbered C311 to C303, C303 to C304, C312 to C305, C304 to C306, C305 to C307, C306 to C308, C307 to C309, C308 to C310, C309 to C311, C310 to C312, R310 to R301, R311 to R302, R313 to R303, R316 to R304, R321 to R305, R322 to R306, R305 to R307, R306 to R308, R307 to R309, R312 to R310, R301 to R311, R315 to R312, R302 to R313, R303 to R314, R304 to R315, R317 to R316, R318 to R317, R319 to R318, R320 to R319, R314 to R320, R308 to R321, R309 to R322, U302 to U301, U303 to U302, U301 to U303

Commit message: Updare pcb
Parts:
- C301, C302, C303, C304, C305, C306, C307, C308, C309, C311, C312: footprint (none) -> Capacitor_SMD:C_0402_1005Metric
- C310: footprint (none) -> Capacitor_SMD:C_Elec_4x5.4; LCSC (none) -> C213487; MPN (none) -> VT1C100M0405
- FB301: footprint (none) -> Inductor_SMD:L_0402_1005Metric; LCSC (none) -> C76883; MPN (none) -> BLM15AG102SN1D
- R301, R302, R303, R304, R305, R306, R307, R308, R309, R310, R311, R312, R313, R314, R315, R316, R317, R318, R319, R320, R321, R322: footprint (none) -> Resistor_SMD:R_0402_1005Metric
Changed lines of the file:
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@@
 			)
 		)
-		(property "Footprint" ""
+		(property "Footprint" "Resistor_SMD:R_0402_1005Metric"
 			(at 139.7 78.74 0)
 			(effects
@@
 			)
 		)
-		(property "Footprint" ""
+		(property "Footprint" "Resistor_SMD:R_0402_1005Metric"
 			(at 45.72 102.87 0)
 			(effects
@@
 			)
 		)
-		(property "Footprint" ""
+		(property "Footprint" "Resistor_SMD:R_0402_1005Metric"
 			(at 215.9 102.87 0)
 			(effects
@@
 			)
 		)
-		(property "Footprint" ""
+		(property "Footprint" "Resistor_SMD:R_0402_1005Metric"
 			(at 127 78.74 0)
 			(effects
@@
 			)
 		)
-		(property "Footprint" ""
+		(property "Footprint" "Capacitor_SMD:C_0402_1005Metric"
 			(at 203.2 38.1 0)
 			(effects
@@
 			)
 		)
-		(property "Footprint" ""
+		(property "Footprint" "Capacitor_SMD:C_0402_1005Metric"
 			(at 135.89 36.83 0)
 			(effects
@@
 			)
 		)
-		(property "Footprint" ""
+		(property "Footprint" "Resistor_SMD:R_0402_1005Metric"
 			(at 146.05 78.74 0)
 			(effects
@@
 			)
 		)
-		(property "Footprint" ""
+		(property "Footprint" "Capacitor_SMD:C_0402_1005Metric"
 			(at 62.23 36.83 0)
 			(effects
@@
 			)
 		)
-		(property "Footprint" ""
+		(property "Footprint" "Resistor_SMD:R_0402_1005Metric"
 			(at 133.35 78.74 0)
 			(effects
@@
 			)
 		)
-		(property "Footprint" ""
+		(property "Footprint" "Capacitor_SMD:C_0402_1005Metric"
 			(at 82.55 135.89 0)
 			(effects
@@
 			)
 		)
-		(property "Footprint" ""
+		(property "Footprint" "Resistor_SMD:R_0402_1005Metric"
 			(at 78.74 93.98 0)
 			(effects
@@
 			)
 		)
-		(property "Footprint" ""
+		(property "Footprint" "Capacitor_SMD:C_0402_1005Metric"
 			(at 72.39 36.83 0)
 			(effects
@@
 			)
 		)
-		(property "Footprint" ""
+		(property "Footprint" "Resistor_SMD:R_0402_1005Metric"
 			(at 273.05 87.63 0)
 			(effects
@@
 			)
 		)
-		(property "Footprint" ""
+		(property "Footprint" "Resistor_SMD:R_0402_1005Metric"
 			(at 234.95 102.87 0)
 			(effects
@@
 			)
 		)
-		(property "Footprint" ""
+		(property "Footprint" "Resistor_SMD:R_0402_1005Metric"
 			(at 228.6 102.87 0)
 			(effects
@@
 			)
 		)
-		(property "Footprint" ""
+		(property "Footprint" "Capacitor_SMD:C_0402_1005Metric"
 			(at 97.79 36.83 0)
 			(effects
@@
 			)
 		)
-		(property "Footprint" ""
+		(property "Footprint" "Resistor_SMD:R_0402_1005Metric"
 			(at 127 99.06 0)
 			(effects
@@
 			)
 		)
-		(property "Footprint" ""
+		(property "Footprint" "Resistor_SMD:R_0402_1005Metric"
 			(at 54.61 85.09 0)
 			(effects
@@
 			)
 		)
-		(property "Footprint" ""
+		(property "Footprint" "Resistor_SMD:R_0402_1005Metric"
 			(at 64.77 85.09 0)
 			(effects
@@
 			)
 		)
-		(property "Footprint" ""
+		(property "Footprint" "Resistor_SMD:R_0402_1005Metric"
 			(at 45.72 113.03 0)
 			(effects
@@
 			)
 		)
-		(property "Footprint" ""
+		(property "Footprint" "Resistor_SMD:R_0402_1005Metric"
 			(at 45.72 88.9 0)
 			(effects
@@
 			)
 		)
-		(property "Footprint" ""
+		(property "Footprint" "Capacitor_SMD:C_0402_1005Metric"
 			(at 110.49 36.83 0)
 			(effects
@@
 			)
 		)
-		(property "Footprint" ""
+		(property "Footprint" "Resistor_SMD:R_0402_1005Metric"
 			(at 275.59 87.63 0)
 			(effects
@@
 			)
 		)
-		(property "Footprint" ""
+		(property "Footprint" "Capacitor_SMD:C_0402_1005Metric"
 			(at 234.95 111.76 0)
 			(effects
@@
 			)
 		)
-		(property "Footprint" ""
+		(property "Footprint" "Resistor_SMD:R_0402_1005Metric"
 			(at 271.78 96.52 0)
 			(effects
@@
 			)
 		)
-		(property "Footprint" ""
+		(property "Footprint" "Resistor_SMD:R_0402_1005Metric"
 			(at 45.72 91.44 0)
 			(effects
@@
 			)
 		)
-		(property "Footprint" ""
+		(property "Footprint" "Resistor_SMD:R_0402_1005Metric"
 			(at 222.25 102.87 0)
 			(effects
@@
 		(on_board yes)
 		(dnp no)
-		(fields_autoplaced yes)
 		(property "Reference" "C310"
 			(at 148.59 35.5662 0)
@@
 			)
 		)
-		(property "Footprint" ""
+		(property "Footprint" "Capacitor_SMD:C_Elec_4x5.4"
 			(at 146.05 36.83 0)
 			(effects
@@
 			)
 		)
-		(property "Datasheet" "~"
+		(property "Datasheet" "https://www.lcsc.com/product-detail/Aluminum-Electrolytic-Capacitors-SMD_ROQANG-VT1C100M0405_C213487.html"
 			(at 146.05 36.83 0)
 			(effects
@@
 			)
 		)
+		(property "MPN" "VT1C100M0405"
+			(at 148.082 43.942 0)
+			(effects
+				(font
+					(size 1.27 1.27)
+				)
+				(hide yes)
+			)
+		)
+		(property "LCSC" " C213487"
+			(at 146.05 36.83 0)
+			(effects
+				(font
+					(size 1.27 1.27)
+				)
+				(hide yes)
+			)
+		)
 		(pin "1"
 		)
@@
 			)
 		)
-		(property "Footprint" ""
+		(property "Footprint" "Inductor_SMD:L_0402_1005Metric"
 			(at 83.82 34.798 90)
 			(effects
@@
 			)
 		)
-		(property "Datasheet" "~"
+		(property "Datasheet" "https://www.lcsc.com/product-detail/span-style-background-color-ff0-Ferrite-span-Beads_Murata-Electronics-BLM15AG102SN1D_C76883.html"
 			(at 83.82 33.02 0)
 			(effects
@@
 			)
 		)
+		(property "MPN" " BLM15AG102SN1D"
+			(at 83.82 33.02 90)
+			(effects
+				(font
+					(size 1.27 1.27)
+				)
+				(hide yes)
+			)
+		)
+		(property "LCSC" "C76883 "
+			(at 83.82 33.02 90)
+			(effects
+				(font
+					(size 1.27 1.27)
+				)
+				(hide yes)
+			)
+		)
 		(pin "2"
 		)
@@
 			)
 		)
-		(property "Footprint" ""
+		(property "Footprint" "Resistor_SMD:R_0402_1005Metric"
 			(at 45.72 96.52 0)
 			(effects
@@
 			)
 		)
-		(property "Footprint" ""
+		(property "Footprint" "Capacitor_SMD:C_0402_1005Metric"
 			(at 66.04 135.89 0)
 			(effects
@@
 			)
 		)
-		(property "Footprint" ""
+		(property "Footprint" "Capacitor_SMD:C_0402_1005Metric"
 			(at 52.07 36.83 0)
 			(effects
@@
 			)
 		)
-		(property "Footprint" ""
+		(property "Footprint" "Resistor_SMD:R_0402_1005Metric"
 			(at 59.69 85.09 0)
 			(effects
@@
 			)
 		)
-		(property "Footprint" ""
+		(property "Footprint" "Capacitor_SMD:C_0402_1005Metric"
 			(at 125.73 36.83 0)
 			(effects
@@
 			)
 		)
-		(property "Footprint" ""
+		(property "Footprint" "Resistor_SMD:R_0402_1005Metric"
 			(at 45.72 109.22 0)
 			(effects

Commit message: create pcb
Parts:
- C303, C305: value 30p -> 20p
Changed lines of the file:
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@@
 			)
 		)
-		(property "Value" "30p"
+		(property "Value" "20p"
 			(at 85.344 135.636 90)
 			(effects
@@
 			)
 		)
-		(property "Value" "30p"
+		(property "Value" "20p"
 			(at 68.834 135.636 90)
 			(effects

Commit message: usb c modif schematic
Parts:
- C312: footprint Capacitor_SMD:C_0402_1005Metric -> Capacitor_SMD:C_1206_3216Metric; LCSC (none) -> C9196; Mfr (none) -> 1206B102K202NT
Changed lines of the file:
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@@
 			)
 		)
-		(property "Footprint" "Capacitor_SMD:C_0402_1005Metric"
+		(property "Footprint" "Capacitor_SMD:C_1206_3216Metric"
 			(at 234.95 111.76 0)
 			(effects
@@
 			)
 		)
-		(property "Datasheet" "~"
+		(property "Datasheet" "https://www.lcsc.com/datasheet/lcsc_datasheet_2304140030_FH--Guangdong-Fenghua-Advanced-Tech-1206B102K202NT_C9196.pdf"
 			(at 234.95 111.76 0)
 			(effects
@@
 			(at 234.95 111.76 0)
 			(effects
+				(font
+					(size 1.27 1.27)
+				)
+				(hide yes)
+			)
+		)
+		(property "Mfr" "1206B102K202NT"
+			(at 234.95 111.76 0)
+			(effects
+				(font
+					(size 1.27 1.27)
+				)
+				(hide yes)
+			)
+		)
+		(property "LCSC" "C9196"
+			(at 234.95 111.76 0)
+			(effects

Commit message: Placement des composants
On va mourir
Parts:
- C310: footprint Capacitor_SMD:C_Elec_4x5.4 -> Capacitor_SMD:C_0402_1005Metric; LCSC C213487 -> C15525; MPN VT1C100M0405 -> CL05A106MQ5NUNC
- C312: footprint Capacitor_SMD:C_1206_3216Metric -> Capacitor_SMD:C_0402_1005Metric; LCSC C9196 -> (none); Mfr 1206B102K202NT -> (none)
Connections:
- net CT: now also C310.2; no longer C310.1
- net GND: now also C310.1; no longer C310.2
Changed lines of the file:
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@@
+	)
+	(symbol
+		(lib_id "Device:C_Small")
+		(at 146.05 36.83 180)
+		(unit 1)
+		(exclude_from_sim no)
+		(in_bom yes)
+		(on_board yes)
+		(dnp no)
+		(property "Reference" "C310"
+			(at 152.4 35.306 0)
+			(effects
+				(font
+					(size 1.27 1.27)
+				)
+				(justify left)
+			)
+		)
+		(property "Value" "10u"
+			(at 151.13 38.1 0)
+			(effects
+				(font
+					(size 1.27 1.27)
+				)
+				(justify left)
+			)
+		)
+		(property "Footprint" "Capacitor_SMD:C_0402_1005Metric"
+			(at 146.05 36.83 0)
+			(effects
+				(font
+					(size 1.27 1.27)
+				)
+				(hide yes)
+			)
+		)
+		(property "Datasheet" "https://www.lcsc.com/datasheet/lcsc_datasheet_2208231630_Samsung-Electro-Mechanics-CL05A106MQ5NUNC_C15525.pdf"
+			(at 146.05 36.83 0)
+			(effects
+				(font
+					(size 1.27 1.27)
+				)
+				(hide yes)
+			)
+		)
+		(property "Description" "Unpolarized capacitor, small symbol"
+			(at 146.05 36.83 0)
+			(effects
+				(font
+					(size 1.27 1.27)
+				)
+				(hide yes)
+			)
+		)
+		(property "MPN" "CL05A106MQ5NUNC"
+			(at 144.018 29.718 0)
+			(effects
+				(font
+					(size 1.27 1.27)
+				)
+				(hide yes)
+			)
+		)
+		(property "LCSC" "C15525"
+			(at 146.05 36.83 0)
+			(effects
+				(font
+					(size 1.27 1.27)
+				)
+				(hide yes)
+			)
+		)
+		(pin "1"
+		)
+		(pin "2"
+		)
+		(instances
+			(project "FabOS_MB"
+				(path "/09377d5d-727f-4ff4-92c8-7a0483d23f1e/97c1e665-4fec-464e-b9f4-4fa619e0ae43"
+					(reference "C310")
+					(unit 1)
+				)
+			)
+		)
 	)
 	(symbol
@@
 			)
 		)
-		(property "Footprint" "Capacitor_SMD:C_1206_3216Metric"
+		(property "Footprint" "Capacitor_SMD:C_0402_1005Metric"
 			(at 234.95 111.76 0)
 			(effects
@@
 			)
 		)
-		(property "Datasheet" "https://www.lcsc.com/datasheet/lcsc_datasheet_2304140030_FH--Guangdong-Fenghua-Advanced-Tech-1206B102K202NT_C9196.pdf"
+		(property "Datasheet" "~"
 			(at 234.95 111.76 0)
 			(effects
@@
 		)
 		(property "Ref ST" "TC1206KKX7RDBB102"
-			(at 234.95 111.76 0)
-			(effects
-				(font
-					(size 1.27 1.27)
-				)
-				(hide yes)
-			)
-		)
-		(property "Mfr" "1206B102K202NT"
-			(at 234.95 111.76 0)
-			(effects
-				(font
-					(size 1.27 1.27)
-				)
-				(hide yes)
-			)
-		)
-		(property "LCSC" "C9196"
 			(at 234.95 111.76 0)
 			(effects
@@
 					(unit 1)
 				)
-			)
-		)
-	)
-	(symbol
-		(lib_id "Device:C_Small")
-		(at 146.05 36.83 0)
-		(unit 1)
-		(exclude_from_sim no)
-		(in_bom yes)
-		(on_board yes)
-		(dnp no)
-		(property "Reference" "C310"
-			(at 148.59 35.5662 0)
-			(effects
-				(font
-					(size 1.27 1.27)
-				)
-				(justify left)
-			)
-		)
-		(property "Value" "10u"
-			(at 148.59 38.1062 0)
-			(effects
-				(font
-					(size 1.27 1.27)
-				)
-				(justify left)
-			)
-		)
-		(property "Footprint" "Capacitor_SMD:C_Elec_4x5.4"
-			(at 146.05 36.83 0)
-			(effects
-				(font
-					(size 1.27 1.27)
-				)
-				(hide yes)
-			)
-		)
-		(property "Datasheet" "https://www.lcsc.com/product-detail/Aluminum-Electrolytic-Capacitors-SMD_ROQANG-VT1C100M0405_C213487.html"
-			(at 146.05 36.83 0)
-			(effects
-				(font
-					(size 1.27 1.27)
-				)
-				(hide yes)
-			)
-		)
-		(property "Description" "Unpolarized capacitor, small symbol"
-			(at 146.05 36.83 0)
-			(effects
-				(font
-					(size 1.27 1.27)
-				)
-				(hide yes)
-			)
-		)
-		(property "MPN" "VT1C100M0405"
-			(at 148.082 43.942 0)
-			(effects
-				(font
-					(size 1.27 1.27)
-				)
-				(hide yes)
-			)
-		)
-		(property "LCSC" " C213487"
-			(at 146.05 36.83 0)
-			(effects
-				(font
-					(size 1.27 1.27)
-				)
-				(hide yes)
-			)
-		)
-		(pin "1"
-		)
-		(pin "2"
-		)
-		(instances
-			(project "FabOS_MB"
-				(path "/09377d5d-727f-4ff4-92c8-7a0483d23f1e/97c1e665-4fec-464e-b9f4-4fa619e0ae43"
-					(reference "C310")
-					(unit 1)
-				)

Commit message: update librairies
Parts:
- Y301: footprint Librairie_MB:Oscillateur crystal 4p -> Crystal:Crystal_SMD_3225-4Pin_3.2x2.5mm
Changed lines of the file:
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@@
 			)
 		)
-		(property "Footprint" "Librairie_MB:Oscillateur crystal 4p"
+		(property "Footprint" "Crystal:Crystal_SMD_3225-4Pin_3.2x2.5mm"
 			(at 74.93 132.08 0)
 			(effects
