File: hardware/FabOS_MB/FabOS_MB.kicad_pcb (KiCad board)
At the start: 4 copper layers, 68 x 68 mm, 114 parts, among them J201 USB_A, J301 RJ45, J401 USB_C_Receptacle, J601 Conn_ST_STDC14, SW601 boot, SW602 SW_Push, SW603 SW_Push, SW604 SW_Push, SW605 SW_Push, U201 NCV7329, U301 LAN8742A, U302 CND-tek B1601S, U401 USBLC6-2SC6, U501 TDPOWER TAS12-5-W2, U502 TPS563201, U601 STM32F407VETx, Y301 Crystal_GND24

Commit message: petit cleanup
Parts:
- moved LED3 6.79 mm to (146.8, 97.2)
- moved R610 6.79 mm to (146.8, 99.1)
- moved LED2 3.98 mm to (150.6, 97.2)
- moved R608 3.98 mm to (150.6, 99.1)
- moved LED1 1.04 mm to (154.6, 97.2)
- moved R606 1.04 mm to (154.6, 99.1)
- renumbered SW603 to BTN1, SW604 to BTN2, SW605 to BTN3, SW601 to Boot, D601 to LED1, D602 to LED2, D603 to LED3, SW602 to RST
Routing:
- net GND: track 48.6 -> 45.0 mm, vias 99 -> 98
- net /STM32/LED3: track 13.1 -> 10.3 mm
- net /STM32/LED2: track 12.7 -> 10.3 mm

Commit message: update_pcb
Routing:
- net /STM32/LED3: track 10.3 -> 18.9 mm
- net /STM32/LED2: track 10.3 -> 15.3 mm
- net /STM32/LED1: track 12.5 -> 13.6 mm
Other:
- board text added: "ESD Protection"
- board text added: "ST LINK"
Changed lines of the file:
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@@
 			(at -2.78 -1.002 0)
 			(layer "F.SilkS")
+			(hide yes)
 			(effects
 				(font
@@
 		(tags "diode")
 		(property "Reference" "D505"
-			(at -2.94 1.002 0)
+			(at 0.05 -0.95 0)
 			(layer "F.SilkS")
+			(hide yes)
 			(effects
 				(font
@@
 		(tags "SOD-323")
 		(property "Reference" "D501"
-			(at 0 -1.85 90)
+			(at 0.05 2.05 90)
 			(layer "F.SilkS")
+			(hide yes)
 			(effects
 				(font
@@
 			(layer "F.Fab")
 		)
-		(fp_text user "${REFERENCE}"
-			(at 0 -1.85 90)
-			(layer "F.Fab")
-			(effects
-				(font
-					(size 1 1)
-					(thickness 0.15)
-				)
-			)
-		)
 		(pad "1" smd roundrect
 			(at -1.05 0 90)
@@
 			(layer "F.SilkS")
 		)
-		(fp_text user "${REFERENCE}"
-			(at 5.8 1.55 90)
-			(unlocked yes)
-			(layer "F.Fab")
-			(effects
-				(font
-					(size 1 1)
-					(thickness 0.15)
-				)
-			)
-		)
 		(pad "1" smd roundrect
 			(at 0 0 90)
@@
 		(tags "capacitor")
 		(property "Reference" "C504"
-			(at 0 -1.16 90)
+			(at 0.1 1.325 -90)
 			(layer "F.SilkS")
+			(hide yes)
 			(effects
 				(font
@@
 		(tags "resistor")
 		(property "Reference" "R501"
-			(at 0 -1.17 90)
+			(at 1.5 -1.775 -90)
 			(layer "F.SilkS")
+			(hide yes)
 			(effects
 				(font
@@
 			(at 0.941 1.637 -90)
 			(layer "F.SilkS")
+			(hide yes)
 			(effects
 				(font
@@
 		(tags "resistor")
 		(property "Reference" "R503"
-			(at 0 -1.17 90)
+			(at 1.45 0.875 90)
 			(layer "F.SilkS")
+			(hide yes)
 			(effects
 				(font
@@
 		)
 		(property ki_fp_filters "MountingHole*Pad*")
-		(sheetname "Root")
+		(sheetname "Racine")
 		(sheetfile "FabOS_MB.kicad_sch")
 		(attr exclude_from_pos_files exclude_from_bom)
@@
 		(tags "resistor")
 		(property "Reference" "R502"
-			(at 0 -1.17 90)
+			(at 1.35 -1.575 90)
 			(layer "F.SilkS")
+			(hide yes)
 			(effects
 				(font
@@
 		)
 		(property ki_fp_filters "MountingHole*Pad*")
-		(sheetname "Root")
+		(sheetname "Racine")
 		(sheetfile "FabOS_MB.kicad_sch")
 		(attr exclude_from_pos_files exclude_from_bom)
@@
 		(tags "diode")
 		(property "Reference" "D503"
-			(at 0.489 -1.951 0)
+			(at 0 -1.25 180)
 			(layer "F.SilkS")
+			(hide yes)
 			(effects
 				(font
@@
 		(tags "capacitor")
 		(property "Reference" "C501"
-			(at 0 -1.16 0)
+			(at 2.775 -0.6 0)
 			(layer "F.SilkS")
+			(hide yes)
 			(effects
 				(font
@@
 		(tags "resistor")
 		(property "Reference" "R504"
-			(at -0.758 1.062 0)
+			(at 0.19 1.25 90)
 			(layer "F.SilkS")
+			(hide yes)
 			(effects
 				(font
@@
 		)
 		(property ki_fp_filters "MountingHole*Pad*")
-		(sheetname "Root")
+		(sheetname "Racine")
 		(sheetfile "FabOS_MB.kicad_sch")
 		(attr exclude_from_pos_files exclude_from_bom)
@@
 			(at 0.0625 -5.118 0)
 			(layer "F.SilkS")
+			(hide yes)
 			(effects
 				(font
@@
 		(tags "inductor")
 		(property "Reference" "L501"
-			(at 0 -1.9 0)
+			(at -0.025 1.9 0)
 			(layer "F.SilkS")
 			(effects
@@
 			(at 0.179 -2.348 180)
 			(layer "F.SilkS")
+			(hide yes)
 			(effects
 				(font
@@
 		(tags "Tactile Switch")
 		(property "Reference" "RST"
-			(at 2.713 2.449 180)
+			(at -0.1 2.2 -90)
 			(layer "F.SilkS")
 			(effects
@@
 		)
 		(property ki_fp_filters "MountingHole*Pad*")
-		(sheetname "Root")
+		(sheetname "Racine")
 		(sheetfile "FabOS_MB.kicad_sch")
 		(attr exclude_from_pos_files exclude_from_bom)
@@
 			(at 0 -1.43 90)
 			(layer "F.SilkS")
+			(hide yes)
 			(effects
 				(font
@@
 			(at -1.901 -1.288 0)
 			(layer "F.SilkS")
+			(hide yes)
 			(effects
 				(font
@@
 			(at 0 -1.43 90)
 			(layer "F.SilkS")
+			(hide yes)
 			(effects
 				(font
@@
 			(at 0.417 -1.21 0)
 			(layer "F.SilkS")
+			(hide yes)
 			(effects
 				(font
@@
 			(at 0 -5.505 0)
 			(layer "F.SilkS")
+			(hide yes)
 			(effects
 				(font
@@
 			(at 2.857 -0.578 0)
 			(layer "F.SilkS")
+			(hide yes)
 			(effects
 				(font
@@
 		(tags "diode")
 		(property "Reference" "D504"
-			(at -0.019 1.415 0)
+			(at -0.2 -0.9 0)
 			(layer "F.SilkS")
+			(hide yes)
 			(effects
 				(font
@@
 		(layer "Edge.Cuts")
 	)
+	(gr_text "ESD\nProtection"
+		(at 103.65 152.6 90)
+		(layer "F.SilkS")
+		(effects
+			(font
+				(size 1 1)
+				(thickness 0.15)
+			)
+		)
+	)
+	(gr_text "ST LINK"
+		(at 97.65 136.25 0)
+		(layer "F.SilkS")
+		(effects
+			(font
+				(size 1 1)
+				(thickness 0.15)
+			)
+			(justify left bottom)
+		)
+	)
 	(segment
 		(start 108.35 152.4)
@@
 	)
 	(segment
-		(start 155.6 102.6)
-		(end 155.6 99.61)
+		(start 158.947 105.947)
+		(end 153.85 100.85)
 		(width 0.15)
 		(layer "F.Cu")
@@
 	)
 	(segment
-		(start 158.947 105.947)
-		(end 155.6 102.6)
+		(start 153.85 100.85)
+		(end 153.85 100.277)
+		(width 0.15)
+		(layer "F.Cu")
+		(net 79)
+	)
+	(segment
+		(start 153.85 100.277)
+		(end 154.559 99.568)
 		(width 0.15)
 		(layer "F.Cu")
@@
 	)
 	(segment
-		(start 158.67 106.061738)
-		(end 154.6 101.991738)
+		(start 158.67 110.645)
+		(end 158.67 106.061738)
 		(width 0.15)
 		(layer "F.Cu")
@@
 	)
 	(segment
-		(start 158.67 110.645)
-		(end 158.67 106.061738)
+		(start 152.180262 99.572)
+		(end 150.622 99.572)
 		(width 0.15)
 		(layer "F.Cu")
@@
 	)
 	(segment
-		(start 158.393 109.728184)
-		(end 158.393 106.176476)
+		(start 158.67 106.061738)
+		(end 152.180262 99.572)
+		(width 0.15)
+		(layer "F.Cu")
+		(net 81)
+	)
+	(segment
+		(start 149.37 99.57)
+		(end 146.812 99.57)
 		(width 0.15)
 		(layer "F.Cu")
@@
 	(segment
 		(start 158.393 106.176476)
-		(end 154.323 102.106476)
+		(end 152.416524 100.2)
 		(width 0.15)
 		(layer "F.Cu")
@@
 	)
 	(segment
-		(start 158.17 109.951184)
-		(end 158.393 109.728184)
+		(start 152.416524 100.2)
+		(end 150 100.2)
 		(width 0.15)
 		(layer "F.Cu")
@@
 		(width 0.15)
 		(layer "F.Cu")
+		(net 82)
+	)
+	(segment
+		(start 158.393 109.728184)
+		(end 158.393 106.176476)
+		(width 0.15)
+		(layer "F.Cu")
+		(net 82)
+	)
+	(segment
+		(start 150 100.2)
+		(end 149.37 99.57)
+		(width 0.15)
+		(layer "F.Cu")
+		(net 82)
+	)
+	(segment
+		(start 158.17 109.951184)
+		(end 158.393 109.728184)
+		(width 0.15)
+		(layer "F.Cu")

Commit message: update pcb
Parts:
- R606, R608, R610: value R_Small -> 1k5
- renumbered LED1 to D601, LED2 to D602, LED3 to D603, Boot to SW601, RST to SW602, BTN1 to SW603, BTN2 to SW604, BTN3 to SW605
Routing:
- net +3.3V: track 47.1 -> 48.1 mm
- net Net-(U502-VFB): track 2.16 -> 2.99 mm
- net GND: vias 98 -> 326
- added copper zone on F.Cu, net Net-(U502-VFB)

Commit message: Update_Pcb
Routing:
- net /STM32/NRST: track 93.4 -> 92.6 mm
- net GND: vias 326 -> 324
- removed copper zone on B.Cu, net GND
- removed copper zone on F.Cu, net GND
Other:
- board text added: "3V3"
- board text added: "BOOT"
- board text added: "BTN1"
- board text added: "BTN2"
- board text added: "BTN3"
- board text added: "FLYBACK"
- board text added: "LED1"
- board text added: "LED2"
- board text added: "LED3"
- board text added: "NRST"
- board text added: "USB"

Commit message: Fab'Rice
Parts:
- added G***: LOGO, LOGO, B.Cu at (132.1, 124.5)

Commit message: update pcb
Other:
- board text added: "L"
- board text added: "LIN"
- board text added: "N"
Changed lines of the file:
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@@
 		(tags "phoenix_contact connector MC_01x03_G_5.08mm")
 		(property "Reference" "e501"
-			(at 5.08 -3.4 0)
+			(at 5.025 2.9325 0)
 			(layer "F.SilkS")
 			(effects
@@
 		)
 	)
+	(gr_text "L"
+		(at 153.3 151.6 0)
+		(layer "F.SilkS" knockout)
+		(effects
+			(font
+				(size 1.5 1.5)
+				(thickness 0.3)
+				(bold yes)
+			)
+			(justify top)
+		)
+	)
 	(gr_text "BOOT"
 		(at 99.9 147.6 90)
@@
 		)
 	)
+	(gr_text "N"
+		(at 148.15 151.55 0)
+		(layer "F.SilkS" knockout)
+		(effects
+			(font
+				(size 1.5 1.5)
+				(thickness 0.3)
+				(bold yes)
+			)
+			(justify top)
+		)
+	)
 	(gr_text "ST LINK"
 		(at 97.2 136.3 0)
@@
 			)
 		)
+	)
+	(gr_text "LIN"
+		(at 148.3 146 0)
+		(layer "F.SilkS" knockout)
+		(effects
+			(font
+				(size 1.5 1.5)
+				(thickness 0.3)
+				(bold yes)
+			)
+		)

Commit message: create gerbers, drills, XY placement files
Routing:
- added copper zone on B.Cu, net GND
- added copper zone on F.Cu, net GND
Other:
- board text added: "DFU"
- board text added: "Rev 1.0 03/07/2024"
- board text added: "|SN : |"
- board text removed: "ESD Protection"
Changed lines of the file:
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@@
 			(disableapertmacros no)
 			(usegerberextensions no)
-			(usegerberattributes yes)
-			(usegerberadvancedattributes yes)
+			(usegerberattributes no)
+			(usegerberadvancedattributes no)
 			(creategerberjobfile yes)
 			(dashed_line_dash_ratio 12.000000)
@@
 			(viasonmask no)
 			(mode 1)
-			(useauxorigin no)
+			(useauxorigin yes)
 			(hpglpennumber 1)
 			(hpglpenspeed 20)
@@
 			(plotinvisibletext no)
 			(sketchpadsonfab no)
-			(subtractmaskfromsilk no)
+			(subtractmaskfromsilk yes)
 			(outputformat 1)
 			(mirror no)
 			(drillshape 0)
 			(scaleselection 1)
-			(outputdirectory "gerbers/")
+			(outputdirectory "jlcpcb/")
 		)
 	)
@@
 		)
 	)
+	(gr_text "|SN :        |"
+		(at 139.1 132.3 0)
+		(layer "F.SilkS" knockout)
+		(effects
+			(font
+				(size 1.5 1.5)
+				(thickness 0.3)
+				(bold yes)
+			)
+			(justify left bottom)
+		)
+	)
+	(gr_text "Rev 1.0\n03/07/2024"
+		(at 97 107.3 0)
+		(layer "F.SilkS")
+		(effects
+			(font
+				(size 1.3 1.3)
+				(thickness 0.2)
+			)
+			(justify left bottom)
+		)
+	)
 	(gr_text "L"
 		(at 153.3 151.6 0)
@@
 		)
 	)
-	(gr_text "ESD\nProtection"
-		(at 103.65 152.6 90)
+	(gr_text "DFU"
+		(at 105.2 155.6 0)
 		(layer "F.SilkS" knockout)
 		(effects
@@
 		(net 2)
 		(net_name "GND")
-		(layer "In1.Cu")
-		(hatch edge 0.5)
-		(priority 1)
-		(connect_pads yes
-			(clearance 0.5)
-		)
-		(min_thickness 0.25)
-		(filled_areas_thickness no)
-		(fill yes
-			(thermal_gap 0.5)
-			(thermal_bridge_width 0.5)
-		)
-		(polygon
-			(pts
-				(xy 96 96) (xy 164 96) (xy 164 164) (xy 96 164)
-			)
-		)
-	)
-	(zone
-		(net 2)
-		(net_name "GND")
-		(layer "In1.Cu")
+		(layers "F.Cu" "In1.Cu" "B.Cu")
 		(hatch edge 0.5)
 		(priority 3)

Commit message: Update libraries
Parts:
- moved J301 6.45 mm to (104.2, 115.7)
- moved U302 6.12 mm to (122.3, 115.7), turned to 0 degrees
- moved J201 4.40 mm to (159.0, 142.0)
- moved U201 3.33 mm to (148.0, 142.0), turned to 0 degrees
- moved J401 1.66 mm to (108.5, 160.3)
- moved U502 1.65 mm to (110.1, 131.4)
Routing:
- net /ethernet/CT: track 14.5 -> 11.7 mm, vias 9 -> 7
- net /ethernet/TXCT: track 14.4 -> 15.8 mm, vias 0 -> 1
- net /ethernet/RXCT: track 6.98 -> 8.39 mm, vias 0 -> 1
