File: hardware/FabOS_MB/lin.kicad_sch (KiCad schematic)
At the start: 6 parts, among them J201 USB_A, U201 NCV7329

Commit message: update pcb
Parts:
- added C201: 10u, symbol Device:C_Small
- added C202: 100n, symbol Device:C_Small
- renumbered C201 to C203, R203 to R201, R204 to R202, R201 to R203
Connections:
- net 5V: now also R202.1, U201.7 (VBB)
- net GND: now also C201.2, C202.2
- net V_LIN: now also C201.1, C202.1; no longer R202.1, U201.7 (VBB)
Other:
- moved on the sheet: J201, R203

Commit message: update
Connections:
- net V_LIN is gone; now on net 5V: C201.1, C202.1
Changed lines of the file:
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@@
-		)
-	)
-	(hierarchical_label "V_LIN"
-		(shape input)
-		(at 118.11 45.72 180)
-		(fields_autoplaced yes)
-		(effects
-			(font
-				(size 1.27 1.27)
-			)
-			(justify right)
 		)
 	)
@@
 		(fields_autoplaced yes)
 		(effects
+			(font
+				(size 1.27 1.27)
+			)
+			(justify right)
+		)
+	)
+	(hierarchical_label "5V"
+		(shape input)
+		(at 118.11 45.72 180)
+		(fields_autoplaced yes)
+		(effects

Commit message: update
Changed lines of the file:
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@@
+	)
+	(junction
+		(at 204.47 92.71)
+		(diameter 0)
+		(color 0 0 0 0)
 	)
 	(junction
@@
 	(wire
 		(pts
+			(xy 204.47 92.71) (xy 207.01 92.71)
+		)
+		(stroke
+			(width 0)
+			(type default)
+		)
+	)
+	(wire
+		(pts
 			(xy 121.92 53.34) (xy 121.92 54.61)
 		)
@@
 	(wire
 		(pts
-			(xy 203.2 92.71) (xy 207.01 92.71)
+			(xy 203.2 92.71) (xy 204.47 92.71)
 		)
 		(stroke
@@
 					(unit 1)
 				)
+			)
+		)
+	)
+	(symbol
+		(lib_id "power:PWR_FLAG")
+		(at 204.47 92.71 0)
+		(unit 1)
+		(exclude_from_sim no)
+		(in_bom yes)
+		(on_board yes)
+		(dnp no)
+		(fields_autoplaced yes)
+		(property "Reference" "#FLG02"
+			(at 204.47 90.805 0)
+			(effects
+				(font
+					(size 1.27 1.27)
+				)
+				(hide yes)
+			)
+		)
+		(property "Value" "PWR_FLAG"
+			(at 204.47 87.63 0)
+			(effects
+				(font
+					(size 1.27 1.27)
+				)
+			)
+		)
+		(property "Footprint" ""
+			(at 204.47 92.71 0)
+			(effects
+				(font
+					(size 1.27 1.27)
+				)
+				(hide yes)
+			)
+		)
+		(property "Datasheet" "~"
+			(at 204.47 92.71 0)
+			(effects
+				(font
+					(size 1.27 1.27)
+				)
+				(hide yes)
+			)
+		)
+		(property "Description" "Special symbol for telling ERC where power comes from"
+			(at 204.47 92.71 0)
+			(effects
+				(font
+					(size 1.27 1.27)
+				)
+				(hide yes)
+			)
+		)
+		(pin "1"
+		)
+		(instances
+			(project ""
+				(path "/09377d5d-727f-4ff4-92c8-7a0483d23f1e/41adeaf0-86bd-4933-9f09-9c5d1e24eb54"
+					(reference "#FLG02")
+					(unit 1)
+				)

Commit message: led
Parts:
- renumbered R203 to R201, R201 to R202, R202 to R203
Changed lines of the file:
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@@
 		(dnp no)
 		(fields_autoplaced yes)
-		(property "Reference" "#PWR0202"
+		(property "Reference" "#PWR0201"
 			(at 88.9 114.3 0)
 			(effects
@@
 			(project "FabOS_MB"
 				(path "/09377d5d-727f-4ff4-92c8-7a0483d23f1e/41adeaf0-86bd-4933-9f09-9c5d1e24eb54"
-					(reference "#PWR0202")
+					(reference "#PWR0201")
 					(unit 1)
 				)
@@
 		(dnp no)
 		(fields_autoplaced yes)
-		(property "Reference" "#FLG02"
+		(property "Reference" "#FLG0201"
 			(at 204.47 90.805 0)
 			(effects
@@
 			(project ""
 				(path "/09377d5d-727f-4ff4-92c8-7a0483d23f1e/41adeaf0-86bd-4933-9f09-9c5d1e24eb54"
-					(reference "#FLG02")
+					(reference "#FLG0201")
 					(unit 1)
 				)
@@
 		(dnp no)
 		(fields_autoplaced yes)
-		(property "Reference" "R201"
+		(property "Reference" "R202"
 			(at 106.68 86.3599 0)
 			(effects
@@
 			(project "FabOS_MB"
 				(path "/09377d5d-727f-4ff4-92c8-7a0483d23f1e/41adeaf0-86bd-4933-9f09-9c5d1e24eb54"
-					(reference "R201")
+					(reference "R202")
 					(unit 1)
 				)
@@
 		(dnp no)
 		(fields_autoplaced yes)
-		(property "Reference" "#PWR0204"
+		(property "Reference" "#PWR0203"
 			(at 146.05 118.11 0)
 			(effects
@@
 			(project "FabOS_MB"
 				(path "/09377d5d-727f-4ff4-92c8-7a0483d23f1e/41adeaf0-86bd-4933-9f09-9c5d1e24eb54"
-					(reference "#PWR0204")
+					(reference "#PWR0203")
 					(unit 1)
 				)
@@
 		(dnp no)
 		(fields_autoplaced yes)
-		(property "Reference" "#PWR0201"
+		(property "Reference" "#PWR0202"
 			(at 121.92 60.96 0)
 			(effects
@@
 			(project "FabOS_MB"
 				(path "/09377d5d-727f-4ff4-92c8-7a0483d23f1e/41adeaf0-86bd-4933-9f09-9c5d1e24eb54"
-					(reference "#PWR0201")
+					(reference "#PWR0202")
 					(unit 1)
 				)
@@
 		(dnp no)
 		(fields_autoplaced yes)
-		(property "Reference" "R203"
+		(property "Reference" "R201"
 			(at 91.44 101.5999 0)
 			(effects
@@
 			(project "FabOS_MB"
 				(path "/09377d5d-727f-4ff4-92c8-7a0483d23f1e/41adeaf0-86bd-4933-9f09-9c5d1e24eb54"
-					(reference "R203")
+					(reference "R201")
 					(unit 1)
 				)
@@
 		(dnp no)
 		(fields_autoplaced yes)
-		(property "Reference" "#PWR0203"
+		(property "Reference" "#PWR0204"
 			(at 195.58 114.3 0)
 			(effects
@@
 			(project "FabOS_MB"
 				(path "/09377d5d-727f-4ff4-92c8-7a0483d23f1e/41adeaf0-86bd-4933-9f09-9c5d1e24eb54"
-					(reference "#PWR0203")
+					(reference "#PWR0204")
 					(unit 1)
 				)
@@
 		(dnp no)
 		(fields_autoplaced yes)
-		(property "Reference" "R202"
+		(property "Reference" "R203"
 			(at 148.59 97.7899 0)
 			(effects
@@
 			(project "FabOS_MB"
 				(path "/09377d5d-727f-4ff4-92c8-7a0483d23f1e/41adeaf0-86bd-4933-9f09-9c5d1e24eb54"
-					(reference "R202")
-					(unit 1)
-				)
+					(reference "R203")
+					(unit 1)
+				)

Commit message: Updare pcb
Parts:
- C201: footprint (none) -> Capacitor_SMD:C_Elec_4x5.4
- C202: footprint (none) -> Capacitor_SMD:C_0402_1005Metric_Pad0.74x0.62mm_HandSolder
- C203: footprint (none) -> Capacitor_SMD:C_0402_1005Metric
- R201, R202, R203: footprint (none) -> Resistor_SMD:R_0402_1005Metric
Changed lines of the file:
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@@
 			)
 		)
-		(property "Footprint" ""
+		(property "Footprint" "Capacitor_SMD:C_Elec_4x5.4"
 			(at 121.92 49.53 0)
 			(effects
@@
 			)
 		)
-		(property "Footprint" ""
+		(property "Footprint" "Resistor_SMD:R_0402_1005Metric"
 			(at 102.362 87.63 90)
 			(effects
@@
 			)
 		)
-		(property "Footprint" ""
+		(property "Footprint" "Resistor_SMD:R_0402_1005Metric"
 			(at 87.122 102.87 90)
 			(effects
@@
 			)
 		)
-		(property "Footprint" ""
+		(property "Footprint" "Capacitor_SMD:C_0402_1005Metric"
 			(at 146.05 106.68 0)
 			(effects
@@
 			)
 		)
-		(property "Footprint" ""
+		(property "Footprint" "Capacitor_SMD:C_0402_1005Metric_Pad0.74x0.62mm_HandSolder"
 			(at 130.81 49.53 0)
 			(effects
@@
 			)
 		)
-		(property "Footprint" ""
+		(property "Footprint" "Resistor_SMD:R_0402_1005Metric"
 			(at 144.272 99.06 90)
 			(effects

Commit message: create pcb
Parts:
- C202: footprint Capacitor_SMD:C_0402_1005Metric_Pad0.74x0.62mm_HandSolder -> Capacitor_SMD:C_0402_1005Metric
Changed lines of the file:
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@@
 			)
 		)
-		(property "Footprint" "Capacitor_SMD:C_0402_1005Metric_Pad0.74x0.62mm_HandSolder"
+		(property "Footprint" "Capacitor_SMD:C_0402_1005Metric"
 			(at 130.81 49.53 0)
 			(effects

Commit message: Placement des composants
On va mourir
Parts:
- C201: footprint Capacitor_SMD:C_Elec_4x5.4 -> Capacitor_SMD:C_0402_1005Metric; LCSC (none) -> C15525; MPN (none) -> CL05A106MQ5NUNC

Commit message: MàJ BoM dans Kicad
Parts:
- C202: LCSC (none) -> C361203
- C203: LCSC (none) -> C92841
- J201: LCSC C42576 -> C42576
- R201: LCSC (none) -> C409682
- R202: LCSC (none) -> C25744
- R203: LCSC (none) -> C102748
- U201: LCSC C603984 -> C194435
Changed lines of the file:
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@@
+			)
+		)
+		(property "LCSC" "C25744"
+			(at 104.14 87.63 0)
+			(effects
+				(font
+					(size 1.27 1.27)
+				)
+				(hide yes)
 			)
 		)
@@
 			)
 		)
-		(property "LCSC" "  C42576"
+		(property "LCSC" " C42576"
 			(at 195.58 97.79 0)
 			(effects
@@
 			)
 		)
+		(property "LCSC" "C409682"
+			(at 88.9 102.87 0)
+			(effects
+				(font
+					(size 1.27 1.27)
+				)
+				(hide yes)
+			)
+		)
 		(pin "1"
 		)
@@
 			)
 		)
+		(property "LCSC" "C92841"
+			(at 146.05 106.68 0)
+			(effects
+				(font
+					(size 1.27 1.27)
+				)
+				(hide yes)
+			)
+		)
 		(pin "1"
 		)
@@
 			)
 		)
-		(property "LCSC" "C603984 "
+		(property "LCSC" "C194435"
 			(at 125.73 85.09 0)
 			(effects
@@
 			)
 		)
+		(property "LCSC" "C361203 "
+			(at 130.81 49.53 0)
+			(effects
+				(font
+					(size 1.27 1.27)
+				)
+				(hide yes)
+			)
+		)
 		(pin "2"
 		)
@@
 			(at 146.05 99.06 0)
 			(effects
+				(font
+					(size 1.27 1.27)
+				)
+				(hide yes)
+			)
+		)
+		(property "LCSC" "C102748"
+			(at 146.05 99.06 0)
+			(effects
