File: hardware/FabOS_MB/usb_c.kicad_sch (KiCad schematic)
At the start: 4 parts, among them J2 USB_C_Receptacle, U6 USBLC6-2SC6

Commit message: update pcb
Parts:
- renumbered J2 to J401, R26 to R401, R27 to R402, U6 to U401
Other:
- note removed: "Valeurs des résistances prises avec le projet S6. Est-il nécessaire de les changer ? Schéma fait à partir du projet S6"
Changed lines of the file:
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@@
-		)
-	)
-	(text "Valeurs des résistances prises avec le projet S6. Est-il nécessaire de les changer ?\nSchéma fait à partir du projet S6"
-		(exclude_from_sim no)
-		(at 231.648 151.13 0)
-		(effects
-			(font
-				(size 1.27 1.27)
-			)
 		)
 	)
@@
 		(on_board yes)
 		(dnp no)
-		(property "Reference" "J2"
+		(property "Reference" "J401"
 			(at 121.92 65.786 0)
 			(effects
@@
 			(project "FabOS_MB"
 				(path "/09377d5d-727f-4ff4-92c8-7a0483d23f1e/7da4f56f-ad27-4eb1-a317-8d2e7594465d"
-					(reference "J2")
+					(reference "J401")
 					(unit 1)
 				)
@@
 		(on_board yes)
 		(dnp no)
-		(property "Reference" "R26"
-			(at 158.75 74.93 90)
+		(property "Reference" "R401"
+			(at 151.638 73.66 90)
 			(effects
 				(font
@@
 		)
 		(property "Value" "5.1k"
-			(at 158.75 77.47 90)
+			(at 151.892 75.438 90)
 			(effects
 				(font
@@
 			(project "FabOS_MB"
 				(path "/09377d5d-727f-4ff4-92c8-7a0483d23f1e/7da4f56f-ad27-4eb1-a317-8d2e7594465d"
-					(reference "R26")
+					(reference "R401")
 					(unit 1)
 				)
@@
 		(on_board yes)
 		(dnp no)
-		(property "Reference" "R27"
-			(at 158.75 88.9 90)
+		(property "Reference" "R402"
+			(at 151.638 88.9 90)
 			(effects
 				(font
@@
 		)
 		(property "Value" "5.1k"
-			(at 158.75 86.36 90)
+			(at 152.146 87.122 90)
 			(effects
 				(font
@@
 			(project "FabOS_MB"
 				(path "/09377d5d-727f-4ff4-92c8-7a0483d23f1e/7da4f56f-ad27-4eb1-a317-8d2e7594465d"
-					(reference "R27")
+					(reference "R402")
 					(unit 1)
 				)
@@
 		(dnp no)
 		(fields_autoplaced yes)
-		(property "Reference" "#PWR037"
+		(property "Reference" "#PWR0403"
 			(at 118.11 121.92 0)
 			(effects
@@
 			(project "FabOS_MB"
 				(path "/09377d5d-727f-4ff4-92c8-7a0483d23f1e/7da4f56f-ad27-4eb1-a317-8d2e7594465d"
-					(reference "#PWR037")
+					(reference "#PWR0403")
 					(unit 1)
 				)
@@
 		(dnp no)
 		(fields_autoplaced yes)
-		(property "Reference" "#PWR039"
+		(property "Reference" "#PWR0402"
 			(at 184.15 104.14 0)
 			(effects
@@
 			(project "FabOS_MB"
 				(path "/09377d5d-727f-4ff4-92c8-7a0483d23f1e/7da4f56f-ad27-4eb1-a317-8d2e7594465d"
-					(reference "#PWR039")
+					(reference "#PWR0402")
 					(unit 1)
 				)
@@
 		(dnp no)
 		(fields_autoplaced yes)
-		(property "Reference" "#PWR038"
+		(property "Reference" "#PWR0401"
 			(at 161.29 81.28 0)
 			(effects
@@
 			(project "FabOS_MB"
 				(path "/09377d5d-727f-4ff4-92c8-7a0483d23f1e/7da4f56f-ad27-4eb1-a317-8d2e7594465d"
-					(reference "#PWR038")
+					(reference "#PWR0401")
 					(unit 1)
 				)
@@
 		(dnp no)
 		(fields_autoplaced yes)
-		(property "Reference" "U6"
+		(property "Reference" "U401"
 			(at 185.8011 82.55 0)
 			(effects
@@
 			(project "FabOS_MB"
 				(path "/09377d5d-727f-4ff4-92c8-7a0483d23f1e/7da4f56f-ad27-4eb1-a317-8d2e7594465d"
-					(reference "U6")
+					(reference "U401")
 					(unit 1)
 				)

Commit message: update
Changed lines of the file:
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@@
 	)
 	(hierarchical_label "VBUS"
-		(shape input)
+		(shape output)
 		(at 184.15 85.09 90)
 		(fields_autoplaced yes)
@@
 	)
 	(hierarchical_label "VBUS"
-		(shape input)
+		(shape output)
 		(at 137.16 74.93 0)
 		(fields_autoplaced yes)

Commit message: usb c modif schematic
Connections:
- net VBUS: no longer J401.A9 (VBUS), J401.B4 (VBUS), J401.B9 (VBUS)
Changed lines of the file:
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@@
 		(pin "A6"
-		)
-		(pin "A9"
 		)
 		(pin "A4"
@@
 		(pin "B12"
 		)
-		(pin "B4"
-		)
-		(pin "B9"
-		)
 		(pin "A1"

Commit message: re correction usb
Connections:
- net GND: no longer J401.A12 (GND), J401.B1 (GND), J401.B12 (GND)
Changed lines of the file:
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@@
 		(pin "B5"
-		)
-		(pin "A12"
 		)
 		(pin "A6"
@@
 		(pin "A8"
 		)
-		(pin "B1"
-		)
 		(pin "B6"
 		)
-		(pin "B12"
-		)
 		(pin "A1"

Commit message: update components placement
Connections:
- net D+: now also U401.3 (I/O2); no longer U401.1 (I/O1)
- net D-: now also U401.1 (I/O1); no longer U401.3 (I/O2)
- net USB_BOOT_DM: now also U401.6 (I/O1); no longer U401.4 (I/O2)
- net USB_BOOT_DP: now also U401.4 (I/O2); no longer U401.6 (I/O1)
Changed lines of the file:
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@@
 	)
 	(label "D+"
+		(at 173.99 92.71 0)
+		(fields_autoplaced yes)
+		(effects
+			(font
+				(size 1.27 1.27)
+			)
+			(justify left bottom)
+		)
+	)
+	(label "D-"
 		(at 173.99 90.17 0)
 		(fields_autoplaced yes)
@@
 		)
 	)
-	(label "D-"
-		(at 173.99 92.71 0)
-		(fields_autoplaced yes)
-		(effects
-			(font
-				(size 1.27 1.27)
-			)
-			(justify left bottom)
-		)
-	)
-	(hierarchical_label "USB_BOOT_DP"
-		(shape bidirectional)
-		(at 193.04 90.17 0)
-		(fields_autoplaced yes)
-		(effects
-			(font
-				(size 1.27 1.27)
-			)
-			(justify left)
-		)
-	)
 	(hierarchical_label "VBUS"
 		(shape output)
@@
 		)
 	)
-	(hierarchical_label "USB_BOOT_DM"
+	(hierarchical_label "USB_BOOT_DP"
 		(shape bidirectional)
 		(at 193.04 92.71 0)
 		(fields_autoplaced yes)
 		(effects
+			(font
+				(size 1.27 1.27)
+			)
+			(justify left)
+		)
+	)
+	(hierarchical_label "USB_BOOT_DM"
+		(shape bidirectional)
+		(at 193.04 90.17 0)
+		(fields_autoplaced yes)
+		(effects

Commit message: Modification PCB
Connections:
- net USB_BOOT_DM renamed USB_BOOT_D-
- net USB_BOOT_DP renamed USB_BOOT_D+
Changed lines of the file:
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@@
 		)
 	)
-	(hierarchical_label "USB_BOOT_DP"
+	(hierarchical_label "USB_BOOT_D+"
 		(shape bidirectional)
 		(at 193.04 92.71 0)
@@
 		)
 	)
-	(hierarchical_label "USB_BOOT_DM"
+	(hierarchical_label "USB_BOOT_D-"
 		(shape bidirectional)
 		(at 193.04 90.17 0)

Commit message: MàJ BoM dans Kicad
Parts:
- R401, R402: LCSC (none) -> C25905
- U401: LCSC (none) -> C2827654
Changed lines of the file:
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@@
+			)
+		)
+		(property "LCSC" "C25905"
+			(at 149.86 77.47 0)
+			(effects
+				(font
+					(size 1.27 1.27)
+				)
+				(hide yes)
 			)
 		)
@@
 		)
 		(property "Fournisseur" "Sotck"
+			(at 149.86 85.09 0)
+			(effects
+				(font
+					(size 1.27 1.27)
+				)
+				(hide yes)
+			)
+		)
+		(property "LCSC" "C25905"
 			(at 149.86 85.09 0)
 			(effects
@@
 			(at 184.15 90.17 0)
 			(effects
+				(font
+					(size 1.27 1.27)
+				)
+				(hide yes)
+			)
+		)
+		(property "LCSC" "C2827654"
+			(at 184.15 90.17 0)
+			(effects
